Commit message: under development

File: allegro_hand_description/urdf/allegro_hand.xacro (robot description, xacro)
@@ -3,4 +3,4 @@
 <xacro:include filename="$(find allegro_hand_description)/urdf/hand.xacro"/>
 <link name="world"/>
-<xacro:ahand prefix="ahand" parent_link="world" xyz="1.0 0 0.15" rpy="0 0 0" left="1" use_ros_control="true"/>
+<xacro:ahand prefix="ahand" parent_link="world" xyz="1.0 0 0.15" rpy="0 0 0" left="1"/>
 </robot>

File: allegro_hand_description/urdf/allegro_hand_transmission.xacro (robot description, xacro)
@@ -14,15 +14,15 @@
     <xacro:finger_transmission finger="${finger}" dof="3"/>
   </xacro:macro>
-<xacro:macro name="finger_transmission" params="finger dof">
-	    <transmission name="${finger}_dof${dof}_trans">
-			<type>transmission_interface/SimpleTransmission</type>
-			<joint name="${finger}_dof${dof}_joint">
-				<hardwareInterface>EffortJointInterface</hardwareInterface>
-			</joint>
-			<actuator name="${finger}_dof${dof}_motor">
-				<hardwareInterface>EffortJointInterface</hardwareInterface>
-				<mechanicalReduction>1</mechanicalReduction>
-			</actuator>
-	    </transmission>
-</xacro:macro>
+  <xacro:macro name="finger_transmission" params="finger dof">
+	<transmission name="${finger}_dof${dof}_trans">
+		<type>transmission_interface/SimpleTransmission</type>
+		<joint name="${finger}_dof${dof}_joint">
+			<hardwareInterface>hardware_interface/EffortJointInterface</hardwareInterface>
+		</joint>
+		<actuator name="${finger}_dof${dof}_motor">
+			<hardwareInterface>hardware_interface/EffortJointInterface</hardwareInterface>
+			<mechanicalReduction>1</mechanicalReduction>
+		</actuator>
+	</transmission>
+ </xacro:macro>
 </robot>

File: allegro_hand_description/urdf/common.xacro (robot description, xacro)
@@ -43,16 +43,16 @@
      for links.
      -->
-  <macro name="cuboid_inertia_def" params="width height length mass">
-    <inertia ixx="${mass * (height * height + length * length) / 12)}"
-             iyy="${mass * (width * width + length * length) / 12)}"
-             izz="${mass * (width * width + height * height) / 12)}"
+  <xacro:macro name="cuboid_inertia_def" params="width height length mass">
+    <inertia ixx="${mass * (height * height + length * length) / 12}"
+             iyy="${mass * (width * width + length * length) / 12}"
+             izz="${mass * (width * width + height * height) / 12}"
              ixy="0" iyz="0" ixz="0"/>
-  </macro>
+  </xacro:macro>
   <!-- length is along the y-axis! -->
-  <macro name="cylinder_inertia_def" params="radius length mass">
-    <inertia ixx="${mass * (3 * radius * radius + length * length) / 12)}"
-             iyy="${mass * radius* radius / 2)}"
-             izz="${mass * (3 * radius * radius + length * length) / 12)}"
+  <xacro:macro name="cylinder_inertia_def" params="radius length mass">
+    <inertia ixx="${mass * (3 * radius * radius + length * length) / 12}"
+             iyy="${mass * radius* radius / 2}"
+             izz="${mass * (3 * radius * radius + length * length) / 12}"
              ixy="0" iyz="0" ixz="0"/>
-  </macro>
+  </xacro:macro>
 </robot>

File: allegro_hand_description/urdf/hand.xacro (robot description, xacro)
@@ -9,5 +9,5 @@
   <xacro:include filename="$(find allegro_hand_description)/urdf/hand_gazebo.xacro"/>
   <!-- High-leveel hand macro -->
-  <xacro:macro name="ahand" params="parent_link prefix xyz rpy left  use_ros_control">
+  <xacro:macro name="ahand" params="parent_link prefix xyz rpy left">
     <xacro:ahand_palm parent_link="${parent_link}" xyz="${xyz}" rpy="${rpy}" left="${left}"/>
     <xacro:ahand_finger_1 prefix="${prefix}"/>
@@ -15,5 +15,5 @@
     <xacro:ahand_finger_3 prefix="${prefix}"/>
     <xacro:ahand_thumb prefix="${prefix}"/>
-    <xacro:allegro_hand_gazebo name="ahand" use_ros_control="${use_ros_control}"/>
+    <xacro:ahand_gazebo name="ahand"/>
     <xacro:ahand_transmission/>
   </xacro:macro>

File: allegro_hand_description/urdf/hand_gazebo.xacro (robot description, xacro)
@@ -1,49 +1,47 @@
 <?xml version="1.0"?>
 <robot xmlns:xacro="http://ros.org/wiki/xacro">
-	<xacro:macro name="allegro_hand_gazebo" params="name use_ros_control">
-			<xacro:if value="${use_ros_control}">
-				<gazebo>
-					<plugin name="gazebo_ros_control" filename="libgazebo_ros_control.so">
-						<robotNamespace>/${name}</robotNamespace>
-					</plugin>
-				</gazebo>
-			</xacro:if>
-   			<gazebo reference="ahand_palm_link">
-      				<xacro:gz_hand_link collide="false"/>
-    			</gazebo>
-    			<xacro:gazebo_one_finger finger="f1" />
-    			<xacro:gazebo_one_finger finger="f2" />
-    			<xacro:gazebo_one_finger finger="f3" />
-    			<xacro:gazebo_one_finger finger="thumb"/>
+	<xacro:macro name="ahand_gazebo" params="name">
+		<gazebo>
+			<plugin name="${name}_hw_sim" filename="libahand_hw_gazebo_plugin.so">
+				<robotNamespace>/${name}</robotNamespace>
+			</plugin>
+		</gazebo>
+   	<gazebo reference="ahand_palm_link">
+    	<xacro:gz_hand_link collide="false"/>
+    </gazebo>
+    <xacro:gazebo_one_finger finger="f1" />
+    <xacro:gazebo_one_finger finger="f2" />
+    <xacro:gazebo_one_finger finger="f3" />
+    <xacro:gazebo_one_finger finger="thumb"/>
 	</xacro:macro>
-  	<xacro:macro name="gz_hand_link" params="collide">
-    		<mu1>0.05</mu1> <!--  Coefficient of friction. Was 0.8 before but then almost impossible to slip. -->
-    		<mu2>0.05</mu2> <!-- 0.8/ 0.05 -->
-    		<kp>400000</kp> <!-- This defines the springiness of the contacts: 400000 -->
-    		<xacro:if value="${collide}">
-      			<selfCollide>false</selfCollide>
-    		</xacro:if>
-  	</xacro:macro>
-  	<xacro:macro name="gz_joint">
-    		<provideFeedback>true</provideFeedback>
-    		<implicitSpringDamper>true</implicitSpringDamper>
-    		<!--<kp>0.0</kp>[> CFM <]-->
-    		<!--<kd>0.0</kd>[> ERP <]-->
-    		<!--<cfmDamping>true</cfmDamping>-->
-    		<!--<dynamics damping="5.5" friction="1"/>-->
-  	</xacro:macro>
-  	<xacro:macro name="gazebo_one_finger" params="finger">
-    		<xacro:gazebo_finger_segment finger="${finger}" dof="0" collide="false"/>
-    		<xacro:gazebo_finger_segment finger="${finger}" dof="1" collide="false"/>
-    		<xacro:gazebo_finger_segment finger="${finger}" dof="2" collide="false"/>
-    		<xacro:gazebo_finger_segment finger="${finger}" dof="3" collide="false"/>
-  	</xacro:macro>
+	<xacro:macro name="gazebo_one_finger" params="finger">
+  	<xacro:gazebo_finger_segment finger="${finger}" dof="0" collide="false"/>
+    <xacro:gazebo_finger_segment finger="${finger}" dof="1" collide="false"/>
+    <xacro:gazebo_finger_segment finger="${finger}" dof="2" collide="false"/>
+    <xacro:gazebo_finger_segment finger="${finger}" dof="3" collide="false"/>
+  </xacro:macro>
 	<xacro:macro name="gazebo_finger_segment" params="finger dof collide">
 		<gazebo reference="${finger}_dof${dof}_joint">
-      			<xacro:gz_joint/>
-    		</gazebo>
-    		<gazebo reference="${finger}_dof1_link">
-      			<xacro:gz_hand_link collide="${collide}"/>
-    		</gazebo>
+    	<xacro:gz_joint/>
+    </gazebo>
+    <gazebo reference="${finger}_dof${dof}_link">
+    	<xacro:gz_hand_link collide="${collide}"/>
+    </gazebo>
 	</xacro:macro>
+	<xacro:macro name="gz_hand_link" params="collide">
+  	<mu1>0.05</mu1> <!--  Coefficient of friction. Was 0.8 before but then almost impossible to slip. -->
+    <mu2>0.05</mu2> <!-- 0.8/ 0.05 -->
+    <kp>400000</kp> <!-- This defines the springiness of the contacts: 400000 -->
+    <xacro:if value="${collide}">
+    	<selfCollide>false</selfCollide>
+    </xacro:if>
+  </xacro:macro>
+  <xacro:macro name="gz_joint">
+  	<provideFeedback>true</provideFeedback>
+    <implicitSpringDamper>true</implicitSpringDamper>
+    <!--<kp>0.0</kp>[> CFM <]-->
+    <!--<kd>0.0</kd>[> ERP <]-->
+    <!--<cfmDamping>true</cfmDamping>-->
+    <!--<dynamics damping="5.5" friction="1"/>-->
+  </xacro:macro>
 </robot>
