Commit message: fixed loading controller

File: allegro_hand_description/urdf/allegro_hand.xacro (robot description, xacro)
@@ -1,6 +1,8 @@
 <?xml version="1.0"?>
 <robot name="ahand" xmlns:xacro="http://www.ros.org/wiki/xacro">
-<xacro:include filename="$(find allegro_hand_description)/urdf/hand.xacro"/>
-<link name="world"/>
-<xacro:ahand prefix="ahand" parent_link="world" xyz="1.0 0 0.15" rpy="0 0 0" left="1"/>
+<!--xacro:include filename="$(find allegro_hand_description)/urdf/hand.xacro"/-->
+<xacro:include filename="$(find allegro_hand_description)/urdf/allegro_hand_description_right.xacro"/>
+<xacro:ahand_robot name="ahand"/>
+<!--link name="world"/-->
+<!--xacro:ahand prefix="ahand" parent_link="world" xyz="1.0 0 0.15" rpy="0 0 0" left="1"/-->
 </robot>

File: allegro_hand_description/urdf/allegro_hand_description_right.xacro (robot description, xacro)
@@ -45,19 +45,24 @@
     <xacro:property name="limit_3_t_low" value="-0.262"/>
     <!-- ============================================================================= -->
+  <xacro:include filename="$(find allegro_hand_description)/urdf/common.xacro"/>
+  <xacro:property name="b" value="0.02"/> <!-- 0.8 damping // 0.2 ..-->
+  <xacro:property name="c" value="0.8"/> <!-- friction: not used ... -->
   <!-- Include transmissions -->
   <xacro:include filename="$(find allegro_hand_description)/urdf/allegro_hand_transmission.xacro"/>
   <!-- Include Gazebo -->
-  <!--xacro:include filename="$(find allegro_hand_description)/urdf/hand_gazebo.xacro"/-->
+  <xacro:include filename="$(find allegro_hand_description)/urdf/hand_gazebo.xacro"/>
+  <!-- URDF model with default base_link (world)-->
+  <xacro:macro name="ahand_robot" params="name">
     <!-- Base link -->
     <link name="hand_root">
       <origin xyz="0 0 0"/>
     </link>
-    <joint name="root_to_base" type="fixed">
+    <joint name="${name}_root_to_base" type="fixed">
       <parent link="hand_root"/>
-      <child link="palm_link"/>
+      <child link="${name}_palm_link"/>
       <origin xyz="0 0 ${palm_link_z}"/>
     </joint>
     <!-- PALM -->
-    <link name="palm_link">
+    <link name="${name}_palm_link">
         <visual>
             <geometry>
@@ -69,10 +74,10 @@
             </material>
         </visual>
-        <collision>
+        <!--collision>
             <origin rpy="0 0 0" xyz="-0.009300 0 -${palm_link_z/2}"/>
             <geometry>
                 <box size="0.0408 0.1130 ${palm_link_z}"/>
             </geometry>
-        </collision>
+        </collision-->
         <inertial>
           <origin xyz="0 0 ${palm_link_z/2}" rpy="0 0 0"/>
@@ -89,4 +94,5 @@
     <!-- for LEFT HAND switch the sign of the **offset_origin_y** and **finger_angle_r** parameters-->
     <xacro:finger
+	    name="${name}"
             finger_num="0"
             offset_origin_x="${offset_origin_x_const}"
@@ -96,4 +102,5 @@
             />
     <xacro:finger
+	    name="${name}"
             finger_num="1"
             offset_origin_x="${offset_origin_x_const}"
@@ -103,4 +110,5 @@
             />
     <xacro:finger
+	    name="${name}"
             finger_num="2"
             offset_origin_x="${offset_origin_x_const}"
@@ -111,4 +119,5 @@
     <!-- THUMB -->
     <xacro:thumb_right
+	    name="${name}"
             finger_num="3"
             offset_origin_x="-0.0182"
@@ -120,9 +129,11 @@
             />
     <!-- ============================================================================= -->
+    <xacro:ahand_gazebo name="${name}"/>
+    <xacro:ahand_transmission name="${name}"/>
+   </xacro:macro>
     <!-- THUMB MACRO -->
-    <xacro:macro name="thumb_right"
-                 params="finger_num offset_origin_x offset_origin_y offset_origin_z finger_angle_r finger_angle_p finger_angle_y">
+   <xacro:macro name="thumb_right" params="name finger_num offset_origin_x offset_origin_y offset_origin_z finger_angle_r finger_angle_p finger_angle_y">
         <!-- [LINK 12] -->
-        <link name="link_${finger_num*4+0}">
+        <link name="${name}_link_${finger_num*4+0}">
             <visual>
                 <geometry>
@@ -134,10 +145,10 @@
                 <origin rpy="${180*DEG2RAD} 0 0" xyz="0 0 0"/>
             </visual>
-            <collision>
+            <!--collision>
                 <geometry>
                     <box size="${link0_t_x} ${link0_t_y} ${link0_t_z}"/>
                 </geometry>
                 <origin rpy="0 0 0" xyz="${-0.0358/2+0.0} ${.018/2} ${.029/2}"/>
-            </collision>
+            </collision-->
             <inertial>
               <mass value="0.0176" />
@@ -148,17 +159,17 @@
             </inertial>
         </link>
-        <joint name="joint_${finger_num*4+0}" type="revolute">
+        <joint name="${name}_joint_${finger_num*4+0}" type="revolute">
             <axis xyz="-1 0 0"/>
             <limit effort="15" velocity="7"
                    lower="${limit_0_t_low-joint_safety_margin}"
                    upper="${limit_0_t_up-joint_safety_margin}"/>
-            <parent link="palm_link"/>
-            <child link="link_${finger_num*4+0}"/>
+            <parent link="${name}_palm_link"/>
+            <child link="${name}_link_${finger_num*4+0}"/>
             <origin rpy="${finger_angle_r} ${finger_angle_p} ${finger_angle_y}"
                     xyz="${offset_origin_x} ${offset_origin_y} ${offset_origin_z}"/>
-            <dynamics damping="3" friction="10"/>
+              <dynamics damping="${0.1*b}" friction="${0.1*c}"/>
         </joint>
         <!-- [LINK 13] -->
-        <link name="link_${finger_num*4+1}">
+        <link name="${name}_link_${finger_num*4+1}">
             <visual>
                 <geometry>
@@ -169,10 +180,10 @@
                 </material>
             </visual>
-            <collision>
+            <!--collision>
                 <geometry>
                     <box size="${links_x} ${links_y} ${link1_t_z}"/>
                 </geometry>
                 <origin rpy="0 0 0" xyz="0 0 ${link1_t_z/2}"/>
-            </collision>
+            </collision-->
             <inertial>
               <mass value="0.0119" />
@@ -183,16 +194,16 @@
             </inertial>
         </link>
-        <joint name="joint_${finger_num*4+1}" type="revolute">
+        <joint name="${name}_joint_${finger_num*4+1}" type="revolute">
             <axis xyz="0 0 1"/>
             <limit effort="15" velocity="7"
                    lower="${limit_1_t_low+joint_safety_margin}"
                    upper="${limit_1_t_up-joint_safety_margin}"/>
-            <parent link="link_${finger_num*4+0}"/>
-            <child link="link_${finger_num*4+1}"/>
+            <parent link="${name}_link_${finger_num*4+0}"/>
+            <child link="${name}_link_${finger_num*4+1}"/>
             <origin xyz="-0.027 0.005 0.0399"/>
-            <dynamics damping="3" friction="5"/>
+            <dynamics damping="${0.1*b}" friction="${0.1*c}"/>
         </joint>
         <!-- [LINK 14] -->
-        <link name="link_${finger_num*4+2}">
+        <link name="${name}_link_${finger_num*4+2}">
             <visual>
                 <geometry>
@@ -202,10 +213,10 @@
                 </material>
             </visual>
-            <collision>
+            <!--collision>
                 <geometry>
                     <box size="${links_x} ${links_y} ${link2_t_z}"/>
                 </geometry>
                 <origin rpy="0 0 0" xyz="0 0 ${link2_t_z/2}"/>
-            </collision>
+            </collision-->
             <inertial>
               <mass value="0.038" />
@@ -215,16 +226,16 @@
             </inertial>
         </link>
-        <joint name="joint_${finger_num*4+2}" type="revolute">
+        <joint name="${name}_joint_${finger_num*4+2}" type="revolute">
             <axis xyz="0 1 0"/>
             <limit effort="15" velocity="7"
                    lower="${limit_2_t_low+joint_safety_margin}"
                    upper="${limit_2_t_up-joint_safety_margin}"/>
-            <parent link="link_${finger_num*4+1}"/>
-            <child link="link_${finger_num*4+2}"/>
+            <parent link="${name}_link_${finger_num*4+1}"/>
+            <child link="${name}_link_${finger_num*4+2}"/>
             <origin xyz="0 0 ${link1_t_z}"/>
-            <dynamics damping="3" friction="10"/>
+            <dynamics damping="${0.1*b}" friction="${0.1*c}"/>
         </joint>
         <!-- [LINK 15] -->
-        <link name="link_${finger_num*4+3}">
+        <link name="${name}_link_${finger_num*4+3}">
             <visual>
                 <geometry>
@@ -234,10 +245,10 @@
                 </material>
             </visual>
-            <collision>
+            <!--collision>
                 <geometry>
                     <box size="${links_x} ${links_y} ${link3_t_z-fingerTip_r}"/>
                 </geometry>
                 <origin rpy="0 0 0" xyz="0 0 ${(link3_t_z-fingerTip_r)/2}"/>
-            </collision>
+            </collision-->
             <inertial>
               <mass value="0.0388" />
@@ -248,16 +259,16 @@
             </inertial>
         </link>
-        <joint name="joint_${finger_num*4+3}" type="revolute">
+        <joint name="${name}_joint_${finger_num*4+3}" type="revolute">
             <axis xyz="0 1 0"/>
             <limit effort="15" velocity="7"
                    lower="${limit_3_t_low+joint_safety_margin}"
                    upper="${limit_3_t_up-joint_safety_margin}"/>
-            <parent link="link_${finger_num*4+2}"/>
-            <child link="link_${finger_num*4+3}"/>
+            <parent link="${name}_link_${finger_num*4+2}"/>
+            <child link="${name}_link_${finger_num*4+3}"/>
             <origin xyz="0 0 ${link2_t_z}"/>
-            <dynamics damping="3" friction="12"/>
+            <dynamics damping="${0.1*b}" friction="${0.1*c}"/>
         </joint>
         <!-- [FINGER TIP] -->
-        <link name="link_${finger_num*4+3}_tip">
+        <link name="${name}_link_${finger_num*4+3}_tip">
             <visual>
                 <geometry>
@@ -268,10 +279,10 @@
                 </material>
             </visual>
-            <collision>
+            <!--collision>
                 <geometry>
                     <sphere radius="${fingerTip_r}"/>
                 </geometry>
                 <origin rpy="0 0 0" xyz="0 0 0"/>
-            </collision>
+            </collision-->
             <inertial>
               <mass value="0.0168" />
@@ -282,7 +293,7 @@
             </inertial>
         </link>
-        <joint name="joint_${finger_num*4+3}_tip" type="fixed">
-            <parent link="link_${finger_num*4+3}"/>
-            <child link="link_${finger_num*4+3}_tip"/>
+        <joint name="${name}_joint_${finger_num*4+3}_tip" type="fixed">
+            <parent link="${name}_link_${finger_num*4+3}"/>
+            <child link="${name}_link_${finger_num*4+3}_tip"/>
             <origin rpy="0 0 0" xyz="0 0 ${link3_t_z-fingerTip_r}"/>
         </joint>
@@ -290,8 +301,7 @@
     <!-- END THUMB MACRO -->
     <!-- THREE FINGER MACRO -->
-    <xacro:macro name="finger"
-                 params="finger_num offset_origin_x offset_origin_y offset_origin_z finger_angle_r">
+    <xacro:macro name="finger" params="name finger_num offset_origin_x offset_origin_y offset_origin_z finger_angle_r">
         <!-- [LINK 0, 4, 8] -->
-        <link name="link_${finger_num*4+0}">
+        <link name="${name}_link_${finger_num*4+0}">
             <visual>
                 <geometry>
@@ -314,17 +324,17 @@
             </inertial>
         </link>
-        <joint name="joint_${finger_num*4+0}" type="revolute">
+        <joint name="${name}_joint_${finger_num*4+0}" type="revolute">
             <axis xyz="0 0 1"/>
             <limit effort="15" velocity="7"
                    lower="${limit_0_low+joint_safety_margin}"
                    upper="${limit_0_up-joint_safety_margin}"/>
-            <parent link="palm_link"/>
-            <child link="link_${finger_num*4+0}"/>
+            <parent link="${name}_palm_link"/>
+            <child link="${name}_link_${finger_num*4+0}"/>
             <origin rpy="${finger_angle_r} 0 0"
                     xyz="${offset_origin_x} ${offset_origin_y} ${offset_origin_z}"/>
-            <dynamics damping="3" friction="10"/>
+            <dynamics damping="${0.1*b}" friction="${0.1*c}"/>
         </joint>
         <!-- [LINK 1, 5, 9] -->
-        <link name="link_${finger_num*4+1}">
+        <link name="${name}_link_${finger_num*4+1}">
             <visual>
                 <geometry>
@@ -333,10 +343,10 @@
                 <material name="black"/>
             </visual>
-            <collision>
+            <!--collision>
                 <geometry>
                     <box size="${links_x} ${links_y} ${link1_z}"/>
                 </geometry>
                 <origin rpy="0 0 0" xyz="0 0 ${link1_z/2}"/>
-            </collision>
+            </collision-->
             <inertial>
               <mass value="0.065" />
@@ -347,16 +357,16 @@
             </inertial>
         </link>
-        <joint name="joint_${finger_num*4+1}" type="revolute">
+        <joint name="${name}_joint_${finger_num*4+1}" type="revolute">
             <limit effort="15" velocity="7"
                    lower="${limit_1_low+joint_safety_margin}"
                    upper="${limit_1_up-joint_safety_margin}"/>
             <axis xyz="0 1 0"/>
-            <parent link="link_${finger_num*4+0}"/>
-            <child link="link_${finger_num*4+1}"/>
+            <parent link="${name}_link_${finger_num*4+0}"/>
+            <child link="${name}_link_${finger_num*4+1}"/>
             <origin xyz="0 0 ${link0_z}"/>
-            <dynamics damping="3" friction="5"/>
+            <dynamics damping="${0.1*b}" friction="${0.1*c}"/>
         </joint>
         <!-- [LINK 2, 6, 10]-->
-        <link name="link_${finger_num*4+2}">
+        <link name="${name}_link_${finger_num*4+2}">
             <visual>
                 <geometry>
@@ -365,10 +375,10 @@
                 <material name="black"/>
             </visual>
-            <collision>
+            <!--collision>
                 <geometry>
                     <box size="${links_x} ${links_y} ${link2_z}"/>
                 </geometry>
                 <origin rpy="0 0 0" xyz="0 0 ${link2_z/2}"/>
-            </collision>
+            </collision-->
             <inertial>
               <mass value="0.0355" />
@@ -379,16 +389,16 @@
             </inertial>
         </link>
-        <joint name="joint_${finger_num*4+2}" type="revolute">
+        <joint name="${name}_joint_${finger_num*4+2}" type="revolute">
             <axis xyz="0 1 0"/>
             <limit effort="15" velocity="7"
                    lower="${limit_2_low+joint_safety_margin}"
                    upper="${limit_2_up-joint_safety_margin}"/>
-            <parent link="link_${finger_num*4+1}"/>
-            <child link="link_${finger_num*4+2}"/>
+            <parent link="${name}_link_${finger_num*4+1}"/>
+            <child  link="${name}_link_${finger_num*4+2}"/>
             <origin xyz="0 0 ${link1_z}"/>
-            <dynamics damping="8" friction="10"/>
+            <dynamics damping="${0.1*b}" friction="${0.1*c}"/>
         </joint>
         <!-- [LINK 3, 7, 11] -->
-        <link name="link_${finger_num*4+3}">
+        <link name="${name}_link_${finger_num*4+3}">
             <visual>
                 <geometry>
@@ -397,10 +407,10 @@
                 <material name="black"/>
             </visual>
-            <collision>
+            <!--collision>
                 <geometry>
                     <box size="${links_x} ${links_y} ${link3_z-fingerTip_r}"/>
                 </geometry>
                 <origin rpy="0 0 0" xyz="0 0 ${(link3_z-fingerTip_r)/2}"/>
-            </collision>
+            </collision-->
             <inertial>
               <mass value="0.0096" />
@@ -411,16 +421,16 @@
             </inertial>
         </link>
-        <joint name="joint_${finger_num*4+3}" type="revolute">
+        <joint name="${name}_joint_${finger_num*4+3}" type="revolute">
             <axis xyz="0 1 0"/>
             <limit effort="15" velocity="7"
                    lower="${limit_3_low+joint_safety_margin}"
                    upper="${limit_3_up-joint_safety_margin}"/>
-            <parent link="link_${finger_num*4+2}"/>
-            <child link="link_${finger_num*4+3}"/>
+            <parent link="${name}_link_${finger_num*4+2}"/>
+            <child link="${name}_link_${finger_num*4+3}"/>
             <origin xyz="0 0 ${link2_z}"/>
-            <dynamics damping="10" friction="12"/>
+            <dynamics damping="${0.1*b}" friction="${0.1*c}"/>
         </joint>
         <!-- [FINGER TIP] -->
-        <link name="link_${finger_num*4+3}_tip">
+        <link name="${name}_link_${finger_num*4+3}_tip">
             <visual>
                 <geometry>
@@ -431,9 +441,9 @@
                 </material>
             </visual>
-            <collision>
+            <!--collision>
                 <geometry>
                     <sphere radius="${fingerTip_r}"/>
                 </geometry>
-            </collision>
+            </collision-->
             <inertial>
               <mass value="0.0168" />
@@ -444,7 +454,7 @@
             </inertial>
         </link>
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
File: allegro_hand_description/urdf/allegro_hand_transmission.xacro (robot description, xacro)
@@ -1,28 +1,33 @@
 <?xml version="1.0"?>
 <robot xmlns:xacro="http://ros.org/wiki/xacro">
-  <!-- High-leveel hand macro -->
-  <xacro:macro name="ahand_transmission">
-    <xacro:ahand_finger_transmission finger="f1" />
-    <xacro:ahand_finger_transmission finger="f2" />
-    <xacro:ahand_finger_transmission finger="f3" />
-    <xacro:ahand_finger_transmission finger="thumb"/>
-  </xacro:macro>
-  <xacro:macro name="ahand_finger_transmission" params="finger">
-    <xacro:finger_transmission finger="${finger}" dof="0"/>
-    <xacro:finger_transmission finger="${finger}" dof="1"/>
-    <xacro:finger_transmission finger="${finger}" dof="2"/>
-    <xacro:finger_transmission finger="${finger}" dof="3"/>
-  </xacro:macro>
-  <xacro:macro name="finger_transmission" params="finger dof">
-	<transmission name="${finger}_dof${dof}_trans">
-		<type>transmission_interface/SimpleTransmission</type>
-		<joint name="${finger}_dof${dof}_joint">
-			<hardwareInterface>hardware_interface/EffortJointInterface</hardwareInterface>
-		</joint>
-		<actuator name="${finger}_dof${dof}_motor">
-			<hardwareInterface>hardware_interface/EffortJointInterface</hardwareInterface>
-			<mechanicalReduction>1</mechanicalReduction>
-		</actuator>
-	</transmission>
+ <xacro:macro name="ahand_transmission" params="name">
+   <xacro:finger_transmission name="${name}" finger_num="0"/>
+   <xacro:finger_transmission name="${name}" finger_num="1"/>
+   <xacro:finger_transmission name="${name}" finger_num="2"/>
+   <xacro:finger_transmission name="${name}" finger_num="3"/>
+   <xacro:finger_transmission name="${name}" finger_num="4"/>
+   <xacro:finger_transmission name="${name}" finger_num="5"/>
+   <xacro:finger_transmission name="${name}" finger_num="6"/>
+   <xacro:finger_transmission name="${name}" finger_num="7"/>
+   <xacro:finger_transmission name="${name}" finger_num="8"/>
+   <xacro:finger_transmission name="${name}" finger_num="9"/>
+   <xacro:finger_transmission name="${name}" finger_num="10"/>
+   <xacro:finger_transmission name="${name}" finger_num="11"/>
+   <xacro:finger_transmission name="${name}" finger_num="12"/>
+   <xacro:finger_transmission name="${name}" finger_num="13"/>
+   <xacro:finger_transmission name="${name}" finger_num="14"/>
+   <xacro:finger_transmission name="${name}" finger_num="15"/>
+ </xacro:macro>
+ <!-- High-leveel hand macro -->
+ <xacro:macro name="finger_transmission" params="name finger_num">
+   <transmission name="${name}_${finger_num}_trans">
+    <type>transmission_interface/SimpleTransmission</type>
+    <joint name="${name}_joint_${finger_num}">
+       <hardwareInterface>hardware_interface/EffortJointInterface</hardwareInterface>
+    </joint>
+    <actuator name="${name}_${finger_num}_motor">
+       <mechanicalReduction>1</mechanicalReduction>
+     </actuator>
+   </transmission>
  </xacro:macro>
 </robot>

File: allegro_hand_description/urdf/hand.xacro (robot description, xacro)
@@ -1,4 +1,4 @@
 <?xml version="1.0"?>
-<robot name="allegro_hand" xmlns:xacro="http://www.ros.org/wiki/xacro">
+<robot name="ahand" xmlns:xacro="http://www.ros.org/wiki/xacro">
   <xacro:include filename="$(find allegro_hand_description)/urdf/common.xacro"/>
   <xacro:property name="b" value="0.02"/> <!-- 0.8 damping // 0.2 ..-->
