Commit message: fixed loading controller

File: allegro_hand_description/urdf/hand_gazebo.xacro (robot description, xacro)
@@ -1,47 +1,32 @@
 <?xml version="1.0"?>
 <robot xmlns:xacro="http://ros.org/wiki/xacro">
-	<xacro:macro name="ahand_gazebo" params="name">
-		<gazebo>
-			<plugin name="${name}_hw_sim" filename="libahand_hw_gazebo_plugin.so">
-				<robotNamespace>/${name}</robotNamespace>
-			</plugin>
-		</gazebo>
-   	<gazebo reference="ahand_palm_link">
-    	<xacro:gz_hand_link collide="false"/>
-    </gazebo>
-    <xacro:gazebo_one_finger finger="f1" />
-    <xacro:gazebo_one_finger finger="f2" />
-    <xacro:gazebo_one_finger finger="f3" />
-    <xacro:gazebo_one_finger finger="thumb"/>
-	</xacro:macro>
-	<xacro:macro name="gazebo_one_finger" params="finger">
-  	<xacro:gazebo_finger_segment finger="${finger}" dof="0" collide="false"/>
-    <xacro:gazebo_finger_segment finger="${finger}" dof="1" collide="false"/>
-    <xacro:gazebo_finger_segment finger="${finger}" dof="2" collide="false"/>
-    <xacro:gazebo_finger_segment finger="${finger}" dof="3" collide="false"/>
+   <xacro:macro name="ahand_gazebo" params="name">
+	<gazebo>
+	  <plugin name="${name}_hw_sim" filename="libahand_hw_gazebo_plugin.so">
+	    <robotNamespace>${name}</robotNamespace>
+	  </plugin>
+	</gazebo>
+    	<xacro:gz_finger finger_num="0"/>
+    	<xacro:gz_finger finger_num="1"/>
+    	<xacro:gz_finger finger_num="2"/>
+    	<xacro:gz_finger finger_num="3"/>
+    	<xacro:gz_finger finger_num="4"/>
+    	<xacro:gz_finger finger_num="5"/>
+    	<xacro:gz_finger finger_num="6"/>
+    	<xacro:gz_finger finger_num="7"/>
+    	<xacro:gz_finger finger_num="8"/>
+    	<xacro:gz_finger finger_num="9"/>
+    	<xacro:gz_finger finger_num="10"/>
+    	<xacro:gz_finger finger_num="11"/>
+    	<xacro:gz_finger finger_num="12"/>
+    	<xacro:gz_finger finger_num="13"/>
+    	<xacro:gz_finger finger_num="14"/>
+    	<xacro:gz_finger finger_num="15"/>
   </xacro:macro>
-	<xacro:macro name="gazebo_finger_segment" params="finger dof collide">
-		<gazebo reference="${finger}_dof${dof}_joint">
-    	<xacro:gz_joint/>
-    </gazebo>
-    <gazebo reference="${finger}_dof${dof}_link">
-    	<xacro:gz_hand_link collide="${collide}"/>
-    </gazebo>
-	</xacro:macro>
-	<xacro:macro name="gz_hand_link" params="collide">
-  	<mu1>0.05</mu1> <!--  Coefficient of friction. Was 0.8 before but then almost impossible to slip. -->
-    <mu2>0.05</mu2> <!-- 0.8/ 0.05 -->
-    <kp>400000</kp> <!-- This defines the springiness of the contacts: 400000 -->
-    <xacro:if value="${collide}">
+  <xacro:macro name="gz_finger" params="finger_num">
+  <gazebo reference="${name}_link_${finger_num}">
+  	<gravity>true</gravity>
     	<selfCollide>false</selfCollide>
-    </xacro:if>
-  </xacro:macro>
-  <xacro:macro name="gz_joint">
-  	<provideFeedback>true</provideFeedback>
-    <implicitSpringDamper>true</implicitSpringDamper>
-    <!--<kp>0.0</kp>[> CFM <]-->
-    <!--<kd>0.0</kd>[> ERP <]-->
-    <!--<cfmDamping>true</cfmDamping>-->
-    <!--<dynamics damping="5.5" friction="1"/>-->
+  </gazebo>
   </xacro:macro>
 </robot>

Commit message: plugin ins working

File: allegro_hand_description/urdf/allegro_hand.xacro (robot description, xacro)
@@ -1,8 +1,6 @@
 <?xml version="1.0"?>
 <robot name="ahand" xmlns:xacro="http://www.ros.org/wiki/xacro">
-<!--xacro:include filename="$(find allegro_hand_description)/urdf/hand.xacro"/-->
 <xacro:include filename="$(find allegro_hand_description)/urdf/allegro_hand_description_right.xacro"/>
-<xacro:ahand_robot name="ahand"/>
-<!--link name="world"/-->
-<!--xacro:ahand prefix="ahand" parent_link="world" xyz="1.0 0 0.15" rpy="0 0 0" left="1"/-->
+<link name="world"/>
+<xacro:ahand_robot name="ahand" parent_link="world" xyz="0.0 0 0.15" rpy="0 0 0"/>
 </robot>
