Commit message: first commit

File: ahand_description/urdf/ahand_description_right.xacro (robot description, xacro)
@@ -10,4 +10,17 @@
     <xacro:property name="link1_z" value="0.0540"/>
     <xacro:property name="link2_z" value="0.0384"/>
+    <!-- according to http://wiki.wonikrobotics.com/AllegroHandWiki/index.php/Link_Masses -->
+    <xacro:property name="link_0_mass" value="${11.0*0.001}"/>
+    <xacro:property name="link_1_mass" value="${65*0.001}"/>
+    <xacro:property name="link_2_mass" value="${35.5*0.001}"/>
+    <xacro:property name="link_3_mass" value="${9.6*0.001}"/>
+    <xacro:property name="link_tip_mass" value="${16.8*0.001}"/>
+    <xacro:property name="thumb_0_mass" value="${17.6*0.001}"/>
+    <xacro:property name="thumb_1_mass" value="${11.9*0.001}"/>
+    <xacro:property name="thumb_2_mass" value="${38.0*0.001}"/>
+    <xacro:property name="thumb_3_mass" value="${38.8*0.001}"/>
+    <xacro:property name="thumb_tip_mass" value="${16.8*0.001}"/>
+    <xacro:property name="palm_mass" value="${415.4*0.001}"/>
+    <!-- http://wiki.wonikrobotics.com/AllegroHandWiki/index.php/Joint_Dimensions_and_Directions -->
     <!-- full height from joint to tip. when used,
          the radius of the finger tip sphere will be subtracted
@@ -45,11 +58,11 @@
     <xacro:property name="limit_3_t_low" value="-0.262"/>
     <!-- ============================================================================= -->
-  <xacro:include filename="$(find allegro_hand_description)/urdf/common.xacro"/>
+  <xacro:include filename="$(find ahand_description)/urdf/common.xacro"/>
   <xacro:property name="b" value="0.02"/> <!-- 0.8 damping // 0.2 ..-->
   <xacro:property name="c" value="0.8"/> <!-- friction: not used ... -->
   <!-- Include transmissions -->
-  <xacro:include filename="$(find allegro_hand_description)/urdf/allegro_hand_transmission.xacro"/>
+  <xacro:include filename="$(find ahand_description)/urdf/allegro_hand_transmission.xacro"/>
   <!-- Include Gazebo -->
-  <xacro:include filename="$(find allegro_hand_description)/urdf/hand_gazebo.xacro"/>
+  <xacro:include filename="$(find ahand_description)/urdf/hand_gazebo.xacro"/>
   <!-- URDF model with default base_link (world)-->
   <xacro:macro name="ahand_robot" params="name parent_link xyz rpy">
@@ -61,27 +74,18 @@
     <!-- PALM -->
     <link name="${name}_palm_link">
-        <visual>
-            <geometry>
-                <mesh filename="package://allegro_hand_description/meshes/base_link.STL"/>
-            </geometry>
-            <origin rpy="0 0 0" xyz="0 0 0 "/>
-            <material name="black">
-                <color rgba="0.2 0.2 0.2 1"/>
-            </material>
+      <inertial>
+        <origin xyz="0 0 -${palm_link_z/2}" rpy="0 0 0"/>
+        <mass value="1.1644" />
+        <xacro:cuboid_inertia_def width="0.04" height="0.095" length="0.10" mass="1.1644"/>
+      </inertial>
+      <visual>
+        <geometry>
+          <mesh filename="package://ahand_description/meshes/base_link.STL"/>
+        </geometry>
+        <origin rpy="0 0 0" xyz="0 0 0 "/>
+          <material name="black">
+            <color rgba="0.2 0.2 0.2 1"/>
+        </material>
         </visual>
-        <!--collision>
-            <origin rpy="0 0 0" xyz="-0.009300 0 -${palm_link_z/2}"/>
-            <geometry>
-                <box size="0.0408 0.1130 ${palm_link_z}"/>
-            </geometry>
-        </collision-->
-        <inertial>
-          <origin xyz="0 0 ${palm_link_z/2}" rpy="0 0 0"/>
-          <mass value="0.4154"/>
-          <inertia
-              ixx="1e-4" ixy="0.0" ixz="0.0"
-              iyy="1e-4" iyz="0.0"
-              izz="1e-4"/>
-        </inertial>
     </link>
     <!-- ============================================================================= -->
@@ -132,20 +136,19 @@
         <!-- [LINK 12] -->
         <link name="${name}_link_${finger_num*4+0}">
-            <visual>
-                <geometry>
-                    <mesh filename="package://allegro_hand_description/meshes/link_12.0_right.STL"/>
-                </geometry>
-                <material name="black">
-                    <color rgba=".2 .2 .2 1"/>
-                </material>
-                <origin rpy="${180*DEG2RAD} 0 0" xyz="0 0 0"/>
-            </visual>
-            <!--collision>
-                <geometry>
-                    <box size="${link0_t_x} ${link0_t_y} ${link0_t_z}"/>
-                </geometry>
-                <origin rpy="0 0 0" xyz="${-0.0358/2+0.0} ${.018/2} ${.029/2}"/>
-            </collision-->
             <inertial>
+              <origin xyz="${-link0_t_x/2} 0 0"/>
+              <xacro:cuboid_inertia_def width="0.02" height="0.04" length="0.04" mass="${thumb_0_mass}"/>
+              <mass value="${thumb_0_mass}" />
+            </inertial>
+            <visual>
+              <geometry>
+                <mesh filename="package://ahand_description/meshes/link_12.0_right.STL"/>
+              </geometry>
+              <material name="black">
+                <color rgba=".2 .2 .2 1"/>
+              </material>
+              <origin rpy="${180*DEG2RAD} 0 0" xyz="0 0 0"/>
+            </visual>
+            <!--inertial>
               <mass value="0.0176" />
               <origin xyz="0 0 0" rpy="0 0 0"/>
@@ -153,5 +156,5 @@
                        iyy="1.43008213333e-05" iyz="6.8068e-06"
                        izz="1.89273333333e-05" />
-            </inertial>
+            </inertial-->
         </link>
         <joint name="${name}_joint_${finger_num*4+0}" type="revolute">
@@ -164,11 +167,16 @@
             <origin rpy="${finger_angle_r} ${finger_angle_p} ${finger_angle_y}"
                     xyz="${offset_origin_x} ${offset_origin_y} ${offset_origin_z}"/>
-              <dynamics damping="${0.1*b}" friction="${0.1*c}"/>
+            <dynamics damping="${0.1*b}" friction="${0.1*c}"/>
         </joint>
         <!-- [LINK 13] -->
         <link name="${name}_link_${finger_num*4+1}">
-            <visual>
-                <geometry>
-                    <mesh filename="package://allegro_hand_description/meshes/link_13.0.STL"/>
+          <inertial>
+            <origin xyz="0.0 0.0 ${link1_t_z/2} "/>
+            <xacro:cuboid_inertia_def width="0.02" height="0.02" length="0.02" mass="${thumb_1_mass}"/>
+            <mass value="${thumb_1_mass}" />
+          </inertial>
+          <visual>
+                <geometry>
+                    <mesh filename="package://ahand_description/meshes/link_13.0.STL"/>
                 </geometry>
                 <material name="black">
@@ -182,5 +190,5 @@
                 <origin rpy="0 0 0" xyz="0 0 ${link1_t_z/2}"/>
             </collision-->
-            <inertial>
+            <!--inertial>
               <mass value="0.0119" />
               <origin xyz="0 0 0" rpy="0 0 0"/>
@@ -188,5 +196,5 @@
                        iyy="4.52362633333e-06" iyz="1.44808125e-06"
                        izz="4.24250866667e-06" />
-            </inertial>
+            </inertial-->
         </link>
         <joint name="${name}_joint_${finger_num*4+1}" type="revolute">
@@ -202,7 +210,12 @@
         <!-- [LINK 14] -->
         <link name="${name}_link_${finger_num*4+2}">
-            <visual>
-                <geometry>
-                    <mesh filename="package://allegro_hand_description/meshes/link_14.0.STL"/>
+            <inertial>
+                  <origin xyz="0.0 0.0 ${link2_t_z/2}"/>
+                        <xacro:cuboid_inertia_def width="0.02" height="0.02" length="0.02" mass="${thumb_2_mass}"/>
+                  <mass value="${thumb_2_mass}" />
+            </inertial>
+            <visual>
+                <geometry>
+                    <mesh filename="package://ahand_description/meshes/link_14.0.STL"/>
                 </geometry>
                 <material name="black">
@@ -215,10 +228,10 @@
                 <origin rpy="0 0 0" xyz="0 0 ${link2_t_z/2}"/>
             </collision-->
-            <inertial>
+            <!--inertial>
               <mass value="0.038" />
               <origin xyz="0 0 0" rpy="0 0 0"/>
               <inertia ixx="4.30439933333e-05" ixy="9.57068e-06" ixz="5.1205e-06" iyy="1.44451933333e-05"
                        iyz="1.342825e-05" izz="4.30439933333e-05" />
-            </inertial>
+            </inertial-->
         </link>
         <joint name="${name}_joint_${finger_num*4+2}" type="revolute">
@@ -234,7 +247,12 @@
         <!-- [LINK 15] -->
         <link name="${name}_link_${finger_num*4+3}">
-            <visual>
-                <geometry>
-                    <mesh filename="package://allegro_hand_description/meshes/link_15.0.STL"/>
+          <inertial>
+                <origin xyz="0.0 0.0 ${link3_t_z/2}"/>
+                      <xacro:cuboid_inertia_def width="0.02" height="0.02" length="0.02" mass="${thumb_3_mass}"/>
+                <mass value="${thumb_3_mass}" />
+          </inertial>
+          <visual>
+                <geometry>
+                    <mesh filename="package://ahand_description/meshes/link_15.0.STL"/>
                 </geometry>
                 <material name="black">
@@ -247,5 +265,5 @@
                 <origin rpy="0 0 0" xyz="0 0 ${(link3_t_z-fingerTip_r)/2}"/>
             </collision-->
-            <inertial>
+            <!--inertial>
               <mass value="0.0388" />
               <origin xyz="0 0 0" rpy="0 0 0"/>
@@ -253,5 +271,5 @@
                        iyy="1.47493026667e-5" iyz="1.1283525e-5"
                        izz="3.29223173333e-05" />
-            </inertial>
+            </inertial-->
         </link>
         <joint name="${name}_joint_${finger_num*4+3}" type="revolute">
@@ -267,7 +285,12 @@
         <!-- [FINGER TIP] -->
         <link name="${name}_link_${finger_num*4+3}_tip">
-            <visual>
-                <geometry>
-                    <mesh filename="package://allegro_hand_description/meshes/link_15.0_tip.STL"/>
+          <inertial>
+                <origin xyz="0.0 0.0 0.0"/>
+                      <xacro:cuboid_inertia_def width="0.02" height="0.05" length="0.02" mass="${thumb_tip_mass}"/>
+                <mass value="${thumb_tip_mass}" />
+          </inertial>
+            <visual>
+                <geometry>
+                    <mesh filename="package://ahand_description/meshes/link_15.0_tip.STL"/>
                 </geometry>
                 <material name="white">
@@ -281,5 +304,5 @@
                 <origin rpy="0 0 0" xyz="0 0 0"/>
             </collision-->
-            <inertial>
+            <!--inertial>
               <mass value="0.0168" />
               <origin xyz="0 0 0" rpy="0 0 0"/>
@@ -287,5 +310,5 @@
                        iyy="9.68e-07" iyz="0"
                        izz="9.68e-07" />
-            </inertial>
+            </inertial-->
         </link>
         <joint name="${name}_joint_${finger_num*4+3}_tip" type="fixed">
@@ -300,7 +323,12 @@
         <!-- [LINK 0, 4, 8] -->
         <link name="${name}_link_${finger_num*4+0}">
-            <visual>
-                <geometry>
-                    <mesh filename="package://allegro_hand_description/meshes/link_0.0.STL"/>
+            <inertial>
+              <origin xyz="0.00 0 0.01"/>
+              <xacro:cuboid_inertia_def width="0.025" height="0.02" length="0.025" mass="${link_0_mass}"/>
+              <mass value="${link_0_mass}" />
+            </inertial>
+            <visual>
+                <geometry>
+                    <mesh filename="package://ahand_description/meshes/link_0.0.STL"/>
                 </geometry>
                 <material name="black"/>
@@ -312,11 +340,4 @@
                 <origin rpy="0 0 0" xyz="0 0 ${link0_z/2}"/>
             </collision>
-            <inertial>
-              <mass value="0.0119" />
-              <origin xyz="0 0 0" rpy="0 0 0"/>
-              <inertia ixx="1.01666658333e-06" ixy="0.0" ixz="0.0"
-                       iyy="6.47677333333e-07" iyz="0.0"
-                       izz="1.01666658333e-06" />
-            </inertial>
         </link>
         <joint name="${name}_joint_${finger_num*4+0}" type="revolute">
@@ -333,23 +354,21 @@
         <!-- [LINK 1, 5, 9] -->
         <link name="${name}_link_${finger_num*4+1}">
-            <visual>
-                <geometry>
-                    <mesh filename="package://allegro_hand_description/meshes/link_1.0.STL"/>
-                </geometry>
-                <material name="black"/>
-            </visual>
-            <!--collision>
+          <inertial>
+        		<origin xyz="0. 0. ${link1_z/2}" rpy="1.5707 0 0"/>
+        		<xacro:cuboid_inertia_def width="0.025" height="0.054" length="0.025" mass="${link_1_mass}"/>
+        		<mass value="${link_2_mass}" />
+      		</inertial>
+          <visual>
+            <geometry>
+              <mesh filename="package://ahand_description/meshes/link_1.0.STL"/>
+            </geometry>
+            <material name="black"/>
+          </visual>
+          <collision>
                 <geometry>
                     <box size="${links_x} ${links_y} ${link1_z}"/>
                 </geometry>
                 <origin rpy="0 0 0" xyz="0 0 ${link1_z/2}"/>
-            </collision-->
-            <inertial>
-              <mass value="0.065" />
-              <origin xyz="0 0 0" rpy="0 0 0"/>
-              <inertia ixx="7.95654166667e-05" ixy="1.7199e-05" ixz="8.75875e-06"
-                       iyy="2.47088833333e-05" iyz="2.413125e-05"
-                       izz="7.95654166667e-05" />
-            </inertial>
+          </collision>
         </link>
         <joint name="${name}_joint_${finger_num*4+1}" type="revolute">
@@ -367,21 +386,19 @@
             <visual>
                 <geometry>
-                    <mesh filename="package://allegro_hand_description/meshes/link_2.0.STL"/>
+                    <mesh filename="package://ahand_description/meshes/link_2.0.STL"/>
                 </geometry>
                 <material name="black"/>
             </visual>
-            <!--collision>
+            <inertial>
+              <origin xyz="0 0 ${link2_z/2}" rpy="0. 1.5707 0."/>
+              <xacro:cuboid_inertia_def width="0.0384" height="0.025" length="0.025" mass="${link_2_mass}"/>
+              <mass value="${link_2_mass}" />
+            </inertial>
+            <collision>
                 <geometry>
                     <box size="${links_x} ${links_y} ${link2_z}"/>
                 </geometry>
                 <origin rpy="0 0 0" xyz="0 0 ${link2_z/2}"/>
-            </collision-->
-            <inertial>
-              <mass value="0.0355" />
-              <origin xyz="0 0 0" rpy="0 0 0"/>
-              <inertia ixx="2.63979183333e-05" ixy="6.67968e-06" ixz="4.783625e-06"
-                       iyy="1.34948516667e-05" iyz="9.372e-06"
-                       izz="2.63979183333e-05" />
-            </inertial>
+            </collision>
         </link>
         <joint name="${name}_joint_${finger_num*4+2}" type="revolute">
@@ -397,23 +414,21 @@
         <!-- [LINK 3, 7, 11] -->
         <link name="${name}_link_${finger_num*4+3}">
-            <visual>
-                <geometry>
-                    <mesh filename="package://allegro_hand_description/meshes/link_3.0.STL"/>
+            <inertial>
+              <origin xyz=" 0 0 0"/>
+              <xacro:cuboid_inertia_def width="0.02" height="0.025" length="0.025" mass="${link_3_mass}"/>
+              <mass value="${link_3_mass}" />
+            </inertial>
+            <visual>
+                <geometry>
+                    <mesh filename="package://ahand_description/meshes/link_3.0.STL"/>
                 </geometry>
                 <material name="black"/>
             </visual>
-            <!--collision>
+            <collision>
                 <geometry>
                     <box size="${links_x} ${links_y} ${link3_z-fingerTip_r}"/>
                 </geometry>
                 <origin rpy="0 0 0" xyz="0 0 ${(link3_z-fingerTip_r)/2}"/>
-            </collision-->
-            <inertial>
-              <mass value="0.0096" />
-              <origin xyz="0 0 0" rpy="0 0 0"/>
-              <inertia ixx="4.701248e-06" ixy="1.255968e-06" ixz="1.2936e-06"
-                       iyy="3.649312e-06" iyz="1.7622e-06"
-                       izz="4.701248e-06" />
-            </inertial>
+            </collision>
         </link>
         <joint name="${name}_joint_${finger_num*4+3}" type="revolute">
@@ -429,24 +444,17 @@
         <!-- [FINGER TIP] -->
         <link name="${name}_link_${finger_num*4+3}_tip">
-            <visual>
-                <geometry>
-                    <mesh filename="package://allegro_hand_description/meshes/link_3.0_tip.STL"/>
-                </geometry>
-                <material name="white">
-                    <color rgba=".9 .9 .9 1"/>
-                </material>
-            </visual>
-            <!--collision>
-                <geometry>
-                    <sphere radius="${fingerTip_r}"/>
-                </geometry>
-            </collision-->
-            <inertial>
-              <mass value="0.0168" />
-              <origin xyz="0 0 0" rpy="0 0 0"/>
-              <inertia ixx="9.68e-07" ixy="0" ixz="0"
-                       iyy="9.68e-07" iyz="0"
-                       izz="9.68e-07" />
-            </inertial>
+          <inertial>
+            <origin xyz="0 0 0"/>
+            <xacro:cuboid_inertia_def width="0.02" height="0.020" length="0.020" mass="${link_tip_mass}"/>
+            <mass value="${link_tip_mass}"/>
+          </inertial>
+          <visual>
+            <geometry>
+              <mesh filename="package://ahand_description/meshes/link_3.0_tip.STL"/>
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
File: ahand_description/urdf/allegro_hand.xacro (robot description, xacro)
@@ -1,5 +1,5 @@
 <?xml version="1.0"?>
 <robot name="ahand" xmlns:xacro="http://www.ros.org/wiki/xacro">
-<xacro:include filename="$(find allegro_hand_description)/urdf/allegro_hand_description_right.xacro"/>
+<xacro:include filename="$(find ahand_description)/urdf/ahand_description_right.xacro"/>
 <link name="world"/>
 <xacro:ahand_robot name="ahand" parent_link="world" xyz="0.0 0 0.15" rpy="0 0 0"/>

File: ahand_description/urdf/common.xacro (robot description, xacro)
@@ -25,5 +25,5 @@
 <robot xmlns:xacro="http://ros.org/wiki/xacro">
   <!-- Directories -->
-  <xacro:property name="models_path" value="package://allegro_hand_description/meshes" />
+  <xacro:property name="models_path" value="package://ahand_description/meshes" />
   <!-- Constants -->
   <xacro:property name="PI" value="3.1415926535897931" />

File: ahand_description/urdf/hand.xacro (robot description, xacro)
@@ -1,11 +1,11 @@
 <?xml version="1.0"?>
 <robot name="ahand" xmlns:xacro="http://www.ros.org/wiki/xacro">
-  <xacro:include filename="$(find allegro_hand_description)/urdf/common.xacro"/>
+  <xacro:include filename="$(find ahand_description)/urdf/common.xacro"/>
   <xacro:property name="b" value="0.02"/> <!-- 0.8 damping // 0.2 ..-->
   <xacro:property name="c" value="0.8"/> <!-- friction: not used ... -->
   <!-- Include transmissions -->
-  <xacro:include filename="$(find allegro_hand_description)/urdf/allegro_hand_transmission.xacro"/>
+  <xacro:include filename="$(find ahand_description)/urdf/allegro_hand_transmission.xacro"/>
   <!-- Include Gazebo -->
-  <xacro:include filename="$(find allegro_hand_description)/urdf/hand_gazebo.xacro"/>
+  <xacro:include filename="$(find ahand_description)/urdf/hand_gazebo.xacro"/>
   <!-- High-leveel hand macro -->
   <xacro:macro name="ahand" params="parent_link prefix xyz rpy left">

File: ahand_description/urdf/tmp.urdf (robot description, URDF)
Before this commit: robot ahand, 22 links, 21 joints
Links:
- link ahand_link_0: geometry collision box size=0.0196 0.0275 0.0164; visual mesh filename=package://ahand_description/meshes/link_0.0.STL
- link ahand_link_1: geometry visual mesh filename=package://ahand_description/meshes/link_1.0.STL
- link ahand_link_10: geometry visual mesh filename=package://ahand_description/meshes/link_2.0.STL
- link ahand_link_11: geometry visual mesh filename=package://ahand_description/meshes/link_3.0.STL
- link ahand_link_11_tip: geometry visual mesh filename=package://ahand_description/meshes/link_3.0_tip.STL
- link ahand_link_12: geometry visual mesh filename=package://ahand_description/meshes/link_12.0_right.STL
- link ahand_link_13: geometry visual mesh filename=package://ahand_description/meshes/link_13.0.STL
- link ahand_link_14: geometry visual mesh filename=package://ahand_description/meshes/link_14.0.STL
- link ahand_link_15: geometry visual mesh filename=package://ahand_description/meshes/link_15.0.STL
- link ahand_link_15_tip: geometry visual mesh filename=package://ahand_description/meshes/link_15.0_tip.STL
- link ahand_link_2: geometry visual mesh filename=package://ahand_description/meshes/link_2.0.STL
- link ahand_link_3: geometry visual mesh filename=package://ahand_description/meshes/link_3.0.STL
- link ahand_link_3_tip: geometry visual mesh filename=package://ahand_description/meshes/link_3.0_tip.STL
- link ahand_link_4: geometry collision box size=0.0196 0.0275 0.0164; visual mesh filename=package://ahand_description/meshes/link_0.0.STL
- link ahand_link_5: geometry visual mesh filename=package://ahand_description/meshes/link_1.0.STL
- link ahand_link_6: geometry visual mesh filename=package://ahand_description/meshes/link_2.0.STL
- link ahand_link_7: geometry visual mesh filename=package://ahand_description/meshes/link_3.0.STL
- link ahand_link_7_tip: geometry visual mesh filename=package://ahand_description/meshes/link_3.0_tip.STL
- link ahand_link_8: geometry collision box size=0.0196 0.0275 0.0164; visual mesh filename=package://ahand_description/meshes/link_0.0.STL
- link ahand_link_9: geometry visual mesh filename=package://ahand_description/meshes/link_1.0.STL
- link ahand_palm_link: geometry visual mesh filename=package://ahand_description/meshes/base_link.STL
