Commit message: fixed joint salt-paper noise

File: ahand_description/urdf/ahand_description_right.xacro (robot description, xacro)
@@ -40,13 +40,15 @@
     <xacro:property name="link3_t_z" value="0.0543"/>
     <!-- ========================= LIMITS ========================= -->
-    <xacro:property name="joint_safety_margin" value="0.1"/>
+    <xacro:property name="joint_safety_margin" value="0.0"/>
+    <!-- finger limit -->
     <xacro:property name="limit_0_up" value="0.57"/>
     <xacro:property name="limit_0_low" value="-0.57"/>
-    <xacro:property name="limit_1_up" value="1.71"/>
+    <xacro:property name="limit_1_up" value="1.74"/>
     <xacro:property name="limit_1_low" value="-0.296"/>
-    <xacro:property name="limit_2_up" value="1.809"/>
-    <xacro:property name="limit_2_low" value="-0.274"/>
-    <xacro:property name="limit_3_up" value="1.718"/>
-    <xacro:property name="limit_3_low" value=" -0.327"/>
+    <xacro:property name="limit_2_up" value="1.74"/> <!-- 1.809 -->
+    <xacro:property name="limit_2_low" value="-0.28"/>
+    <xacro:property name="limit_3_up" value="1.73"/>
+    <xacro:property name="limit_3_low" value=" -0.28"/>
+    <!-- thumb limit -->
     <xacro:property name="limit_0_t_up" value="1.496"/>
     <xacro:property name="limit_0_t_low" value="0.363"/>

Commit message: pd controller working

File: ahand_description/urdf/ahand_description_right.xacro (robot description, xacro)
@@ -51,6 +51,6 @@
     <xacro:property name="limit_3_low" value=" -0.28"/>
     <!-- thumb limit -->
-    <xacro:property name="limit_0_t_up" value="1.496"/>
-    <xacro:property name="limit_0_t_low" value="0.363"/>
+    <xacro:property name="limit_0_t_up" value="1.57"/>
+    <xacro:property name="limit_0_t_low" value="0.275"/>
     <xacro:property name="limit_1_t_up" value="1.263"/>
     <xacro:property name="limit_1_t_low" value="-0.205"/>

Commit message: under devel

File: ahand_description/urdf/ahand_description_right.xacro (robot description, xacro)
@@ -230,10 +230,4 @@
                 <origin rpy="0 0 0" xyz="0 0 ${link2_t_z/2}"/>
             </collision-->
-            <!--inertial>
-              <mass value="0.038" />
-              <origin xyz="0 0 0" rpy="0 0 0"/>
-              <inertia ixx="4.30439933333e-05" ixy="9.57068e-06" ixz="5.1205e-06" iyy="1.44451933333e-05"
-                       iyz="1.342825e-05" izz="4.30439933333e-05" />
-            </inertial-->
         </link>
         <joint name="${name}_joint_${finger_num*4+2}" type="revolute">

Commit message: gazebo sim working

File: ahand_description/urdf/ahand_description_right.xacro (robot description, xacro)
@@ -11,14 +11,15 @@
     <xacro:property name="link2_z" value="0.0384"/>
     <!-- according to http://wiki.wonikrobotics.com/AllegroHandWiki/index.php/Link_Masses -->
-    <xacro:property name="link_0_mass" value="${11.0*0.001}"/>
-    <xacro:property name="link_1_mass" value="${65*0.001}"/>
-    <xacro:property name="link_2_mass" value="${35.5*0.001}"/>
-    <xacro:property name="link_3_mass" value="${9.6*0.001}"/>
-    <xacro:property name="link_tip_mass" value="${16.8*0.001}"/>
-    <xacro:property name="thumb_0_mass" value="${17.6*0.001}"/>
-    <xacro:property name="thumb_1_mass" value="${11.9*0.001}"/>
-    <xacro:property name="thumb_2_mass" value="${38.0*0.001}"/>
-    <xacro:property name="thumb_3_mass" value="${38.8*0.001}"/>
-    <xacro:property name="thumb_tip_mass" value="${16.8*0.001}"/>
+    <xacro:property name="mass_scale" value="1.0"/>
+    <xacro:property name="link_0_mass" value="${11.0*0.001*mass_scale}"/>
+    <xacro:property name="link_1_mass" value="${65*0.001*mass_scale}"/>
+    <xacro:property name="link_2_mass" value="${35.5*0.001*mass_scale}"/>
+    <xacro:property name="link_3_mass" value="${9.6*0.001*mass_scale}"/>
+    <xacro:property name="link_tip_mass" value="${16.8*0.001*mass_scale}"/>
+    <xacro:property name="thumb_0_mass" value="${17.6*0.001*mass_scale}"/>
+    <xacro:property name="thumb_1_mass" value="${11.9*0.001*mass_scale}"/>
+    <xacro:property name="thumb_2_mass" value="${38.0*0.001*mass_scale}"/>
+    <xacro:property name="thumb_3_mass" value="${38.8*0.001*mass_scale}"/>
+    <xacro:property name="thumb_tip_mass" value="${16.8*0.001*mass_scale}"/>
     <xacro:property name="palm_mass" value="${415.4*0.001}"/>
     <!-- http://wiki.wonikrobotics.com/AllegroHandWiki/index.php/Joint_Dimensions_and_Directions -->
@@ -61,10 +62,10 @@
     <!-- ============================================================================= -->
   <xacro:include filename="$(find ahand_description)/urdf/common.xacro"/>
-  <xacro:property name="b" value="0.02"/> <!-- 0.8 damping // 0.2 ..-->
-  <xacro:property name="c" value="0.8"/> <!-- friction: not used ... -->
+  <xacro:property name="b" value="2.0"/>
+  <xacro:property name="c" value="0.0"/>
   <!-- Include transmissions -->
-  <xacro:include filename="$(find ahand_description)/urdf/allegro_hand_transmission.xacro"/>
+  <xacro:include filename="$(find ahand_description)/urdf/ahand_transmission.xacro"/>
   <!-- Include Gazebo -->
-  <xacro:include filename="$(find ahand_description)/urdf/hand_gazebo.xacro"/>
+  <xacro:include filename="$(find ahand_description)/urdf/ahand_gazebo.xacro"/>
   <!-- URDF model with default base_link (world)-->
   <xacro:macro name="ahand_robot" params="name parent_link xyz rpy">
@@ -152,11 +153,4 @@
               <origin rpy="${180*DEG2RAD} 0 0" xyz="0 0 0"/>
             </visual>
-            <!--inertial>
-              <mass value="0.0176" />
-              <origin xyz="0 0 0" rpy="0 0 0"/>
-              <inertia ixx="1.89273333333e-5" ixy="7.16716e-06" ixz="5.35568e-06"
-                       iyy="1.43008213333e-05" iyz="6.8068e-06"
-                       izz="1.89273333333e-05" />
-            </inertial-->
         </link>
         <joint name="${name}_joint_${finger_num*4+0}" type="revolute">
@@ -169,5 +163,5 @@
             <origin rpy="${finger_angle_r} ${finger_angle_p} ${finger_angle_y}"
                     xyz="${offset_origin_x} ${offset_origin_y} ${offset_origin_z}"/>
-            <dynamics damping="${0.1*b}" friction="${0.1*c}"/>
+            <dynamics damping="${b}" friction="${c}"/>
         </joint>
         <!-- [LINK 13] -->
@@ -186,17 +180,4 @@
                 </material>
             </visual>
-            <!--collision>
-                <geometry>
-                    <box size="${links_x} ${links_y} ${link1_t_z}"/>
-                </geometry>
-                <origin rpy="0 0 0" xyz="0 0 ${link1_t_z/2}"/>
-            </collision-->
-            <!--inertial>
-              <mass value="0.0119" />
-              <origin xyz="0 0 0" rpy="0 0 0"/>
-              <inertia ixx="4.24250866667e-06" ixy="1.032087e-06" ixz="1.603525e-06"
-                       iyy="4.52362633333e-06" iyz="1.44808125e-06"
-                       izz="4.24250866667e-06" />
-            </inertial-->
         </link>
         <joint name="${name}_joint_${finger_num*4+1}" type="revolute">
@@ -208,5 +189,5 @@
             <child link="${name}_link_${finger_num*4+1}"/>
             <origin xyz="-0.027 0.005 0.0399"/>
-            <dynamics damping="${0.1*b}" friction="${0.1*c}"/>
+            <dynamics damping="${b}" friction="${c}"/>
         </joint>
         <!-- [LINK 14] -->
@@ -224,10 +205,10 @@
                 </material>
             </visual>
-            <!--collision>
+            <collision>
                 <geometry>
                     <box size="${links_x} ${links_y} ${link2_t_z}"/>
                 </geometry>
                 <origin rpy="0 0 0" xyz="0 0 ${link2_t_z/2}"/>
-            </collision-->
+            </collision>
         </link>
         <joint name="${name}_joint_${finger_num*4+2}" type="revolute">
@@ -239,5 +220,5 @@
             <child link="${name}_link_${finger_num*4+2}"/>
             <origin xyz="0 0 ${link1_t_z}"/>
-            <dynamics damping="${0.1*b}" friction="${0.1*c}"/>
+            <dynamics damping="${b}" friction="${c}"/>
         </joint>
         <!-- [LINK 15] -->
@@ -255,17 +236,10 @@
                 </material>
             </visual>
-            <!--collision>
-                <geometry>
-                    <box size="${links_x} ${links_y} ${link3_t_z-fingerTip_r}"/>
-                </geometry>
-                <origin rpy="0 0 0" xyz="0 0 ${(link3_t_z-fingerTip_r)/2}"/>
-            </collision-->
-            <!--inertial>
-              <mass value="0.0388" />
-              <origin xyz="0 0 0" rpy="0 0 0"/>
-              <inertia ixx="3.29223173333e-05" ixy="8.042076e-06" ixz="5.2283e-06"
-                       iyy="1.47493026667e-5" iyz="1.1283525e-5"
-                       izz="3.29223173333e-05" />
-            </inertial-->
+            <collision>
+                <geometry>
+                    <box size="${links_x} ${links_y} ${link3_t_z-2.0*fingerTip_r}"/>
+                </geometry>
+                <origin rpy="0 0 0" xyz="0 0 ${(link3_t_z-2.0*fingerTip_r)/2}"/>
+            </collision>
         </link>
         <joint name="${name}_joint_${finger_num*4+3}" type="revolute">
@@ -277,7 +251,7 @@
             <child link="${name}_link_${finger_num*4+3}"/>
             <origin xyz="0 0 ${link2_t_z}"/>
-            <dynamics damping="${0.1*b}" friction="${0.1*c}"/>
-        </joint>
-        <!-- [FINGER TIP] -->
+            <dynamics damping="${b}" friction="${c}"/>
+        </joint>
+        <!-- [FINGER TIP THUMB] -->
         <link name="${name}_link_${finger_num*4+3}_tip">
           <inertial>
@@ -294,17 +268,9 @@
                 </material>
             </visual>
-            <!--collision>
-                <geometry>
-                    <sphere radius="${fingerTip_r}"/>
-                </geometry>
-                <origin rpy="0 0 0" xyz="0 0 0"/>
-            </collision-->
-            <!--inertial>
-              <mass value="0.0168" />
-              <origin xyz="0 0 0" rpy="0 0 0"/>
-              <inertia ixx="9.68e-07" ixy="0" ixz="0"
-                       iyy="9.68e-07" iyz="0"
-                       izz="9.68e-07" />
-            </inertial-->
+            <collision>
+                <geometry>
+                    <mesh filename="package://ahand_description/meshes/link_15.0_tip.STL"/>
+                </geometry>
+            </collision>
         </link>
         <joint name="${name}_joint_${finger_num*4+3}_tip" type="fixed">
@@ -346,5 +312,5 @@
             <origin rpy="${finger_angle_r} 0 0"
                     xyz="${offset_origin_x} ${offset_origin_y} ${offset_origin_z}"/>
-            <dynamics damping="${0.1*b}" friction="${0.1*c}"/>
+            <dynamics damping="${b}" friction="${c}"/>
         </joint>
         <!-- [LINK 1, 5, 9] -->
@@ -376,5 +342,5 @@
             <child link="${name}_link_${finger_num*4+1}"/>
             <origin xyz="0 0 ${link0_z}"/>
-            <dynamics damping="${0.1*b}" friction="${0.1*c}"/>
+            <dynamics damping="${b}" friction="${c}"/>
         </joint>
         <!-- [LINK 2, 6, 10]-->
@@ -406,5 +372,5 @@
             <child  link="${name}_link_${finger_num*4+2}"/>
             <origin xyz="0 0 ${link1_z}"/>
-            <dynamics damping="${0.1*b}" friction="${0.1*c}"/>
+            <dynamics damping="${b}" friction="${c}"/>
         </joint>
         <!-- [LINK 3, 7, 11] -->
@@ -423,7 +389,7 @@
             <collision>
                 <geometry>
-                    <box size="${links_x} ${links_y} ${link3_z-fingerTip_r}"/>
-                </geometry>
-                <origin rpy="0 0 0" xyz="0 0 ${(link3_z-fingerTip_r)/2}"/>
+                    <box size="${links_x} ${links_y} ${link3_z-2.0*fingerTip_r}"/>
+                </geometry>
+                <origin rpy="0 0 0" xyz="0 0 ${(link3_z-2.0*fingerTip_r)/2}"/>
             </collision>
         </link>
@@ -436,21 +402,26 @@
             <child link="${name}_link_${finger_num*4+3}"/>
             <origin xyz="0 0 ${link2_z}"/>
-            <dynamics damping="${0.1*b}" friction="${0.1*c}"/>
+            <dynamics damping="${b}" friction="${c}"/>
         </joint>
         <!-- [FINGER TIP] -->
         <link name="${name}_link_${finger_num*4+3}_tip">
-          <inertial>
-            <origin xyz="0 0 0"/>
-            <xacro:cuboid_inertia_def width="0.02" height="0.020" length="0.020" mass="${link_tip_mass}"/>
-            <mass value="${link_tip_mass}"/>
-          </inertial>
-          <visual>
-            <geometry>
-              <mesh filename="package://ahand_description/meshes/link_3.0_tip.STL"/>
-            </geometry>
-            <material name="white">
-              <color rgba=".9 .9 .9 1"/>
-            </material>
-          </visual>
+            <inertial>
+                <origin xyz="0 0 0"/>
+                <xacro:cuboid_inertia_def width="0.02" height="0.020" length="0.020" mass="${link_tip_mass}"/>
+                <mass value="${link_tip_mass}"/>
+            </inertial>
+            <visual>
+                <geometry>
+                    <mesh filename="package://ahand_description/meshes/link_3.0_tip.STL"/>
+                </geometry>
+                <material name="white">
+                    <color rgba=".9 .9 .9 1"/>
+                </material>
+            </visual>
+            <collision>
+                <geometry>
+                    <mesh filename="package://ahand_description/meshes/link_3.0_tip.STL"/>
+                </geometry>
+            </collision>
         </link>
         <joint name="${name}_joint_${finger_num*4+3}_tip" type="fixed">

File: ahand_description/urdf/ahand_gazebo.xacro (robot description, xacro)
@@ -27,5 +27,9 @@
   <gazebo reference="${name}_link_${finger_num}">
   	<gravity>true</gravity>
-    	<selfCollide>false</selfCollide>
+    <selfCollide>false</selfCollide>
+	  <velocity_decay>
+		  <linear>0.2</linear>
+		  <angular>0.4</angular>
+	  </velocity_decay>
   </gazebo>
   </xacro:macro>

Commit message: under devel

File: ahand_description/urdf/ahand_description_right.xacro (robot description, xacro)
@@ -323,5 +323,5 @@
           <visual>
             <geometry>
-              <mesh filename="package://ahand_description/meshes/link_1.0.STL"/>
+              <mesh filename="package://ahand_description/meshes/link_1.dae"/>
             </geometry>
             <material name="black"/>

Commit message: fixed meshes for color in gazebo

File: ahand_description/urdf/ahand_description_right.xacro (robot description, xacro)
@@ -84,5 +84,5 @@
       <visual>
         <geometry>
-          <mesh filename="package://ahand_description/meshes/base_link.STL"/>
+          <mesh filename="package://ahand_description/meshes/base_link.dae"/>
         </geometry>
         <origin rpy="0 0 0" xyz="0 0 0 "/>
@@ -146,5 +146,5 @@
             <visual>
               <geometry>
-                <mesh filename="package://ahand_description/meshes/link_12.0_right.STL"/>
+                <mesh filename="package://ahand_description/meshes/link_12_right.dae"/>
               </geometry>
               <material name="black">
@@ -174,5 +174,5 @@
           <visual>
                 <geometry>
-                    <mesh filename="package://ahand_description/meshes/link_13.0.STL"/>
+                    <mesh filename="package://ahand_description/meshes/link_13.dae"/>
                 </geometry>
                 <material name="black">
@@ -200,5 +200,5 @@
             <visual>
                 <geometry>
-                    <mesh filename="package://ahand_description/meshes/link_14.0.STL"/>
+                    <mesh filename="package://ahand_description/meshes/link_14.dae"/>
                 </geometry>
                 <material name="black">
@@ -231,5 +231,5 @@
           <visual>
                 <geometry>
-                    <mesh filename="package://ahand_description/meshes/link_15.0.STL"/>
+                    <mesh filename="package://ahand_description/meshes/link_15.dae"/>
                 </geometry>
                 <material name="black">
@@ -292,5 +292,5 @@
             <visual>
                 <geometry>
-                    <mesh filename="package://ahand_description/meshes/link_0.0.STL"/>
+                    <mesh filename="package://ahand_description/meshes/link_0.dae"/>
                 </geometry>
                 <material name="black"/>
@@ -348,5 +348,5 @@
             <visual>
                 <geometry>
-                    <mesh filename="package://ahand_description/meshes/link_2.0.STL"/>
+                    <mesh filename="package://ahand_description/meshes/link_2.dae"/>
                 </geometry>
                 <material name="black"/>
@@ -383,5 +383,5 @@
             <visual>
                 <geometry>
-                    <mesh filename="package://ahand_description/meshes/link_3.0.STL"/>
+                    <mesh filename="package://ahand_description/meshes/link_3.dae"/>
                 </geometry>
                 <material name="black"/>
@@ -413,5 +413,5 @@
             <visual>
                 <geometry>
-                    <mesh filename="package://ahand_description/meshes/link_3.0_tip.STL"/>
+                    <mesh filename="package://ahand_description/meshes/link_3_tip.STL"/>
                 </geometry>
                 <material name="white">
@@ -421,5 +421,5 @@
             <collision>
                 <geometry>
-                    <mesh filename="package://ahand_description/meshes/link_3.0_tip.STL"/>
+                    <mesh filename="package://ahand_description/meshes/link_3_tip.STL"/>
                 </geometry>
             </collision>

Commit message: under develop

File: ahand_description/urdf/ahand_description_right.xacro (robot description, xacro)
@@ -62,5 +62,5 @@
     <!-- ============================================================================= -->
   <xacro:include filename="$(find ahand_description)/urdf/common.xacro"/>
-  <xacro:property name="b" value="2.0"/>
+  <xacro:property name="b" value="0.2"/>
   <xacro:property name="c" value="0.0"/>
   <!-- Include transmissions -->
