Commit message: changed link directions

File: ahand_description/urdf/ahand_description_right.xacro (robot description, xacro)
@@ -194,10 +194,11 @@
         <link name="${name}_link_${finger_num*4+2}">
             <inertial>
-                  <origin xyz="0.0 0.0 ${link2_t_z/2}"/>
+                  <origin xyz="${link2_t_z/2} 0.0 0.0"/>
                         <xacro:cuboid_inertia_def width="0.02" height="0.02" length="0.02" mass="${thumb_2_mass}"/>
                   <mass value="${thumb_2_mass}" />
             </inertial>
             <visual>
-                <geometry>
+            	<origin xyz="0 0 0" rpy="${90*DEG2RAD} 0 ${90*DEG2RAD}"/>
+		<geometry>
                     <mesh filename="package://ahand_description/meshes/link_14.dae"/>
                 </geometry>
@@ -209,9 +210,9 @@
                     <box size="${links_x} ${links_y} ${link2_t_z}"/>
                 </geometry>
-                <origin rpy="0 0 0" xyz="0 0 ${link2_t_z/2}"/>
+                <origin rpy="${90*DEG2RAD} 0 ${90*DEG2RAD}" xyz="${link2_t_z/2} 0 0"/>
             </collision>
         </link>
         <joint name="${name}_joint_${finger_num*4+2}" type="revolute">
-            <axis xyz="0 1 0"/>
+            <axis xyz="0 0 1"/>
             <limit effort="15" velocity="7"
                    lower="${limit_2_t_low+joint_safety_margin}"
@@ -219,5 +220,5 @@
             <parent link="${name}_link_${finger_num*4+1}"/>
             <child link="${name}_link_${finger_num*4+2}"/>
-            <origin xyz="0 0 ${link1_t_z}"/>
+            <origin xyz="0 0 ${link1_t_z}" rpy="0 -${90*DEG2RAD} -${90*DEG2RAD}"/>
             <dynamics damping="${b}" friction="${c}"/>
         </joint>
@@ -225,9 +226,10 @@
         <link name="${name}_link_${finger_num*4+3}">
           <inertial>
-                <origin xyz="0.0 0.0 ${link3_t_z/2}"/>
+                <origin xyz="${link3_t_z/2} 0.0 0.0"/>
                       <xacro:cuboid_inertia_def width="0.02" height="0.02" length="0.02" mass="${thumb_3_mass}"/>
                 <mass value="${thumb_3_mass}" />
           </inertial>
           <visual>
+            	<origin xyz="0 0 0" rpy="${90*DEG2RAD} 0 ${90*DEG2RAD}"/>
                 <geometry>
                     <mesh filename="package://ahand_description/meshes/link_15.dae"/>
@@ -240,9 +242,9 @@
                     <box size="${links_x} ${links_y} ${link3_t_z-2.0*fingerTip_r}"/>
                 </geometry>
-                <origin rpy="0 0 0" xyz="0 0 ${(link3_t_z-2.0*fingerTip_r)/2}"/>
+                <origin rpy="${90*DEG2RAD} 0 ${90*DEG2RAD}" xyz="${(link3_t_z-2.0*fingerTip_r)/2} 0 0"/>
             </collision>
         </link>
         <joint name="${name}_joint_${finger_num*4+3}" type="revolute">
-            <axis xyz="0 1 0"/>
+            <axis xyz="0 0 1"/>
             <limit effort="15" velocity="7"
                    lower="${limit_3_t_low+joint_safety_margin}"
@@ -250,5 +252,5 @@
             <parent link="${name}_link_${finger_num*4+2}"/>
             <child link="${name}_link_${finger_num*4+3}"/>
-            <origin xyz="0 0 ${link2_t_z}"/>
+            <origin xyz="${link2_t_z} 0 0" rpy="0 0 0"/>
             <dynamics damping="${b}" friction="${c}"/>
         </joint>
@@ -261,4 +263,5 @@
           </inertial>
             <visual>
+                <origin xyz="0 0 0" rpy="${90*DEG2RAD} 0 ${90*DEG2RAD}"/>
                 <geometry>
                     <mesh filename="package://ahand_description/meshes/link_15.0_tip.STL"/>
@@ -269,4 +272,5 @@
             </visual>
             <collision>
+                <origin xyz="0 0 0" rpy="${90*DEG2RAD} 0 ${90*DEG2RAD}"/>
                 <geometry>
                     <mesh filename="package://ahand_description/meshes/link_15.0_tip.STL"/>
@@ -277,5 +281,5 @@
             <parent link="${name}_link_${finger_num*4+3}"/>
             <child link="${name}_link_${finger_num*4+3}_tip"/>
-            <origin rpy="0 0 0" xyz="0 0 ${link3_t_z-fingerTip_r}"/>
+            <origin rpy="0 0 0" xyz="${link3_t_z-fingerTip_r} 0 0"/>
         </joint>
     </xacro:macro>
@@ -317,9 +321,10 @@
         <link name="${name}_link_${finger_num*4+1}">
           <inertial>
-        		<origin xyz="0. 0. ${link1_z/2}" rpy="1.5707 0 0"/>
-        		<xacro:cuboid_inertia_def width="0.025" height="0.054" length="0.025" mass="${link_1_mass}"/>
-        		<mass value="${link_2_mass}" />
-      		</inertial>
+        	<origin xyz="${link1_z/2} 0. 0." rpy="0 0 1.5707"/>
+        	<xacro:cuboid_inertia_def width="0.025" height="0.054" length="0.025" mass="${link_1_mass}"/>
+        	<mass value="${link_2_mass}" />
+      	  </inertial>
           <visual>
+            <origin xyz="0 0 0" rpy="${90*DEG2RAD} 0 ${90*DEG2RAD}"/>
             <geometry>
               <mesh filename="package://ahand_description/meshes/link_1.dae"/>
@@ -331,5 +336,5 @@
                     <box size="${links_x} ${links_y} ${link1_z}"/>
                 </geometry>
-                <origin rpy="0 0 0" xyz="0 0 ${link1_z/2}"/>
+                <origin xyz="${link1_z/2} 0 0" rpy="${90*DEG2RAD} 0 ${90*DEG2RAD}"/>
           </collision>
         </link>
@@ -338,32 +343,33 @@
                    lower="${limit_1_low+joint_safety_margin}"
                    upper="${limit_1_up-joint_safety_margin}"/>
-            <axis xyz="0 1 0"/>
+            <axis xyz="0 0 1"/>
             <parent link="${name}_link_${finger_num*4+0}"/>
             <child link="${name}_link_${finger_num*4+1}"/>
-            <origin xyz="0 0 ${link0_z}"/>
+            <origin rpy="${90*DEG2RAD} -${90*DEG2RAD} 0" xyz="0 0 ${link0_z}"/>
             <dynamics damping="${b}" friction="${c}"/>
         </joint>
         <!-- [LINK 2, 6, 10]-->
         <link name="${name}_link_${finger_num*4+2}">
-            <visual>
-                <geometry>
-                    <mesh filename="package://ahand_description/meshes/link_2.dae"/>
-                </geometry>
-                <material name="black"/>
-            </visual>
-            <inertial>
-              <origin xyz="0 0 ${link2_z/2}" rpy="0. 1.5707 0."/>
+	    <inertial>
+              <origin xyz="${link2_z/2} 0 0" rpy="0. 0. 0."/>
               <xacro:cuboid_inertia_def width="0.0384" height="0.025" length="0.025" mass="${link_2_mass}"/>
               <mass value="${link_2_mass}" />
             </inertial>
+    	    <visual>
+                <origin xyz="0 0 0" rpy="${90*DEG2RAD} 0 ${90*DEG2RAD}"/>
+                <geometry>
+                    <mesh filename="package://ahand_description/meshes/link_2.dae"/>
+                </geometry>
+                <material name="black"/>
+            </visual>
             <collision>
                 <geometry>
                     <box size="${links_x} ${links_y} ${link2_z}"/>
                 </geometry>
-                <origin rpy="0 0 0" xyz="0 0 ${link2_z/2}"/>
+                <origin xyz="${link2_z/2} 0 0" rpy="${90*DEG2RAD} 0 ${90*DEG2RAD}"/>
             </collision>
         </link>
         <joint name="${name}_joint_${finger_num*4+2}" type="revolute">
-            <axis xyz="0 1 0"/>
+            <axis xyz="0 0 1"/>
             <limit effort="15" velocity="7"
                    lower="${limit_2_low+joint_safety_margin}"
@@ -371,5 +377,5 @@
             <parent link="${name}_link_${finger_num*4+1}"/>
             <child  link="${name}_link_${finger_num*4+2}"/>
-            <origin xyz="0 0 ${link1_z}"/>
+            <origin xyz="${link1_z} 0 0"/>
             <dynamics damping="${b}" friction="${c}"/>
         </joint>
@@ -377,9 +383,10 @@
         <link name="${name}_link_${finger_num*4+3}">
             <inertial>
-              <origin xyz=" 0 0 0"/>
+              <origin xyz=" 0 0 0" rpy="0. 0. 0."/>
               <xacro:cuboid_inertia_def width="0.02" height="0.025" length="0.025" mass="${link_3_mass}"/>
               <mass value="${link_3_mass}" />
             </inertial>
             <visual>
+                <origin xyz="0 0 0" rpy="${90*DEG2RAD} 0 ${90*DEG2RAD}"/>
                 <geometry>
                     <mesh filename="package://ahand_description/meshes/link_3.dae"/>
@@ -391,9 +398,9 @@
                     <box size="${links_x} ${links_y} ${link3_z-2.0*fingerTip_r}"/>
                 </geometry>
-                <origin rpy="0 0 0" xyz="0 0 ${(link3_z-2.0*fingerTip_r)/2}"/>
+                <origin xyz="${(link3_z-2.0*fingerTip_r)/2} 0 0" rpy="${90*DEG2RAD} 0 ${90*DEG2RAD}"/>
             </collision>
         </link>
         <joint name="${name}_joint_${finger_num*4+3}" type="revolute">
-            <axis xyz="0 1 0"/>
+            <axis xyz="0 0 1"/>
             <limit effort="15" velocity="7"
                    lower="${limit_3_low+joint_safety_margin}"
@@ -401,5 +408,5 @@
             <parent link="${name}_link_${finger_num*4+2}"/>
             <child link="${name}_link_${finger_num*4+3}"/>
-            <origin xyz="0 0 ${link2_z}"/>
+            <origin xyz="${link2_z} 0 0"/>
             <dynamics damping="${b}" friction="${c}"/>
         </joint>
@@ -412,4 +419,5 @@
             </inertial>
             <visual>
+                <origin xyz="0 0 0" rpy="0 ${90*DEG2RAD} 0"/>
                 <geometry>
                     <mesh filename="package://ahand_description/meshes/link_3_tip.STL"/>
@@ -420,4 +428,5 @@
             </visual>
             <collision>
+                <origin xyz="0 0 0" rpy="${90*DEG2RAD} 0 ${90*DEG2RAD}"/>
                 <geometry>
                     <mesh filename="package://ahand_description/meshes/link_3_tip.STL"/>
@@ -428,5 +437,5 @@
             <parent link="${name}_link_${finger_num*4+3}"/>
             <child link="${name}_link_${finger_num*4+3}_tip"/>
-            <origin rpy="0 0 0" xyz="0 0 ${link3_z-fingerTip_r}"/>
+            <origin rpy="0 0 0" xyz="${link3_z-fingerTip_r} 0 0"/>
         </joint>
     </xacro:macro>

Commit message: changed thumb FR

File: ahand_description/urdf/ahand_description_right.xacro (robot description, xacro)
@@ -216,5 +216,5 @@
         </link>
         <joint name="${name}_joint_${finger_num*4+2}" type="revolute">
-            <axis xyz="0 0 1"/>
+            <axis xyz="0 0 -1"/>
             <limit effort="15" velocity="7"
                    lower="${limit_2_t_low+joint_safety_margin}"
@@ -222,5 +222,5 @@
             <parent link="${name}_link_${finger_num*4+1}"/>
             <child link="${name}_link_${finger_num*4+2}"/>
-            <origin xyz="0 0 ${link1_t_z}" rpy="0 -${90*DEG2RAD} -${90*DEG2RAD}"/>
+            <origin xyz="0 0 ${link1_t_z}" rpy="${180*DEG2RAD} -${90*DEG2RAD} -${90*DEG2RAD}"/>
             <dynamics damping="${b}" friction="${c}"/>
         </joint>
@@ -248,5 +248,5 @@
         </link>
         <joint name="${name}_joint_${finger_num*4+3}" type="revolute">
-            <axis xyz="0 0 1"/>
+            <axis xyz="0 0 -1"/>
             <limit effort="15" velocity="7"
                    lower="${limit_3_t_low+joint_safety_margin}"
@@ -297,4 +297,5 @@
             </inertial>
             <visual>
+                <origin xyz="0 0 0" rpy="0 0 -${90*DEG2RAD}"/>
                 <geometry>
                     <mesh filename="package://ahand_description/meshes/link_0.dae"/>
@@ -316,6 +317,5 @@
             <parent link="${name}_palm_link"/>
             <child link="${name}_link_${finger_num*4+0}"/>
-            <origin rpy="${finger_angle_r} 0 0"
-                    xyz="${offset_origin_x} ${offset_origin_y} ${offset_origin_z}"/>
+            <origin xyz="${offset_origin_x} ${offset_origin_y} ${offset_origin_z}" rpy="${finger_angle_r} 0 0"/>
             <dynamics damping="${b}" friction="${c}"/>
         </joint>
@@ -328,5 +328,5 @@
       	  </inertial>
           <visual>
-            <origin xyz="0 0 0" rpy="${90*DEG2RAD} 0 ${90*DEG2RAD}"/>
+            <origin xyz="0 0 0" rpy="${90*DEG2RAD} ${180*DEG2RAD} ${90*DEG2RAD}"/>
             <geometry>
               <mesh filename="package://ahand_description/meshes/link_1.dae"/>
@@ -345,8 +345,8 @@
                    lower="${limit_1_low+joint_safety_margin}"
                    upper="${limit_1_up-joint_safety_margin}"/>
-            <axis xyz="0 0 1"/>
+            <axis xyz="0 0 -1"/>
             <parent link="${name}_link_${finger_num*4+0}"/>
             <child link="${name}_link_${finger_num*4+1}"/>
-            <origin rpy="${90*DEG2RAD} -${90*DEG2RAD} 0" xyz="0 0 ${link0_z}"/>
+            <origin xyz="0 0 ${link0_z}" rpy="0 -${90*DEG2RAD} ${90*DEG2RAD}"/>
             <dynamics damping="${b}" friction="${c}"/>
         </joint>
@@ -359,5 +359,5 @@
             </inertial>
     	    <visual>
-                <origin xyz="0 0 0" rpy="${90*DEG2RAD} 0 ${90*DEG2RAD}"/>
+                <origin xyz="0 0 0" rpy="${90*DEG2RAD} ${180*DEG2RAD} ${90*DEG2RAD}"/>
                 <geometry>
                     <mesh filename="package://ahand_description/meshes/link_2.dae"/>
@@ -373,5 +373,5 @@
         </link>
         <joint name="${name}_joint_${finger_num*4+2}" type="revolute">
-            <axis xyz="0 0 1"/>
+            <axis xyz="0 0 -1"/>
             <limit effort="15" velocity="7"
                    lower="${limit_2_low+joint_safety_margin}"
@@ -390,5 +390,5 @@
             </inertial>
             <visual>
-                <origin xyz="0 0 0" rpy="${90*DEG2RAD} 0 ${90*DEG2RAD}"/>
+                <origin xyz="0 0 0" rpy="${90*DEG2RAD} ${180*DEG2RAD} ${90*DEG2RAD}"/>
                 <geometry>
                     <mesh filename="package://ahand_description/meshes/link_3.dae"/>
@@ -404,5 +404,5 @@
         </link>
         <joint name="${name}_joint_${finger_num*4+3}" type="revolute">
-            <axis xyz="0 0 1"/>
+            <axis xyz="0 0 -1"/>
             <limit effort="15" velocity="7"
                    lower="${limit_3_low+joint_safety_margin}"

Commit message: fixed mesh vis

File: ahand_description/urdf/ahand_description_right.xacro (robot description, xacro)
@@ -297,5 +297,5 @@
             </inertial>
             <visual>
-                <origin xyz="0 0 0" rpy="0 0 -${90*DEG2RAD}"/>
+                <origin xyz="0 0 0" rpy="0 0 0"/>
                 <geometry>
                     <mesh filename="package://ahand_description/meshes/link_0.dae"/>
