Commit message: added left and right xacros

File: ahand_description/urdf/ahand.xacro (robot description, xacro)
@@ -1,6 +1,7 @@
 <?xml version="1.0"?>
-<robot name="ahand" xmlns:xacro="http://www.ros.org/wiki/xacro">
-<xacro:include filename="$(find ahand_description)/urdf/ahand_description_right.xacro"/>
-<link name="world"/>
-<xacro:ahand_robot name="ahand" parent_link="world" xyz="0.0 0 0.15" rpy="0 0 0"/>
+<robot name="ahand" xmlns:xacro="http://ros.org/wiki/xacro">
+    <xacro:property name="hand_type" default="left" />
+    <xacro:include filename="$(find ahand_description)/urdf/ahand_${hand_type}.xacro"/>
+    <link name="world"/>
+    <xacro:ahand_robot name="ahand" parent_link="world" xyz="0.0 0 0.15" rpy="0 0 0"/>
 </robot>

File: ahand_description/urdf/ahand_right.xacro (robot description, xacro)
@@ -1,4 +1,4 @@
 <?xml version="1.0"?>
-<robot xmlns:xacro="http://www.ros.org/wiki/xacro" name="allegro_hand_right">
+<robot xmlns:xacro="http://www.ros.org/wiki/xacro" name="ahand_right">
     <xacro:property name="DEG2RAD" value="0.01745329251"/>
     <!-- ======================== BASE PARAMS ========================= -->
@@ -10,18 +10,4 @@
     <xacro:property name="link1_z" value="0.0540"/>
     <xacro:property name="link2_z" value="0.0384"/>
-    <!-- according to http://wiki.wonikrobotics.com/AllegroHandWiki/index.php/Link_Masses -->
-    <xacro:property name="mass_scale" value="1.0"/>
-    <xacro:property name="link_0_mass" value="${11.0*0.001*mass_scale}"/>
-    <xacro:property name="link_1_mass" value="${65*0.001*mass_scale}"/>
-    <xacro:property name="link_2_mass" value="${35.5*0.001*mass_scale}"/>
-    <xacro:property name="link_3_mass" value="${9.6*0.001*mass_scale}"/>
-    <xacro:property name="link_tip_mass" value="${16.8*0.001*mass_scale}"/>
-    <xacro:property name="thumb_0_mass" value="${17.6*0.001*mass_scale}"/>
-    <xacro:property name="thumb_1_mass" value="${11.9*0.001*mass_scale}"/>
-    <xacro:property name="thumb_2_mass" value="${38.0*0.001*mass_scale}"/>
-    <xacro:property name="thumb_3_mass" value="${38.8*0.001*mass_scale}"/>
-    <xacro:property name="thumb_tip_mass" value="${16.8*0.001*mass_scale}"/>
-    <xacro:property name="palm_mass" value="${415.4*0.001}"/>
-    <!-- http://wiki.wonikrobotics.com/AllegroHandWiki/index.php/Joint_Dimensions_and_Directions -->
     <!-- full height from joint to tip. when used,
          the radius of the finger tip sphere will be subtracted
@@ -41,17 +27,15 @@
     <xacro:property name="link3_t_z" value="0.0543"/>
     <!-- ========================= LIMITS ========================= -->
-    <xacro:property name="joint_safety_margin" value="0.0"/>
-    <!-- finger limit -->
+    <xacro:property name="joint_safety_margin" value="0.1"/>
     <xacro:property name="limit_0_up" value="0.57"/>
     <xacro:property name="limit_0_low" value="-0.57"/>
-    <xacro:property name="limit_1_up" value="1.74"/>
+    <xacro:property name="limit_1_up" value="1.71"/>
     <xacro:property name="limit_1_low" value="-0.296"/>
-    <xacro:property name="limit_2_up" value="1.74"/> <!-- 1.809 -->
-    <xacro:property name="limit_2_low" value="-0.28"/>
-    <xacro:property name="limit_3_up" value="1.73"/>
-    <xacro:property name="limit_3_low" value=" -0.28"/>
-    <!-- thumb limit -->
-    <xacro:property name="limit_0_t_up" value="1.57"/>
-    <xacro:property name="limit_0_t_low" value="0.275"/>
+    <xacro:property name="limit_2_up" value="1.809"/>
+    <xacro:property name="limit_2_low" value="-0.274"/>
+    <xacro:property name="limit_3_up" value="1.718"/>
+    <xacro:property name="limit_3_low" value=" -0.327"/>
+    <xacro:property name="limit_0_t_up" value="1.496"/>
+    <xacro:property name="limit_0_t_low" value="0.363"/>
     <xacro:property name="limit_1_t_up" value="1.263"/>
     <xacro:property name="limit_1_t_low" value="-0.205"/>
@@ -61,34 +45,36 @@
     <xacro:property name="limit_3_t_low" value="-0.262"/>
     <!-- ============================================================================= -->
-  <xacro:include filename="$(find ahand_description)/urdf/common.xacro"/>
-  <xacro:property name="b" value="0.2"/>
-  <xacro:property name="c" value="0.0"/>
-  <!-- Include transmissions -->
-  <xacro:include filename="$(find ahand_description)/urdf/ahand_transmission.xacro"/>
-  <!-- Include Gazebo -->
-  <xacro:include filename="$(find ahand_description)/urdf/ahand_gazebo.xacro"/>
-  <!-- URDF model with default base_link (world)-->
-  <xacro:macro name="ahand_robot" params="name parent_link xyz rpy">
+    <!-- Base link -->
+    <xacro:macro name="ahand_robot" params="name parent_link xyz rpy">
     <joint name="${name}_base_joint" type="fixed">
-      <parent link="${parent_link}"/>
-      <child link="${name}_palm_link"/>
-      <origin xyz="${xyz}" rpy="${rpy}"/>
+        <parent link="${parent_link}"/>
+        <child link="${name}_palm_link"/>
+        <origin xyz="${xyz}" rpy="${rpy}"/>
     </joint>
     <!-- PALM -->
     <link name="${name}_palm_link">
-      <inertial>
-        <origin xyz="0 0 -${palm_link_z/2}" rpy="0 0 0"/>
-        <mass value="1.1644" />
-        <xacro:cuboid_inertia_def width="0.04" height="0.095" length="0.10" mass="1.1644"/>
-      </inertial>
-      <visual>
-        <geometry>
-          <mesh filename="package://ahand_description/meshes/base_link.dae"/>
-        </geometry>
-        <origin rpy="0 0 0" xyz="0 0 0 "/>
-          <material name="black">
-            <color rgba="0.2 0.2 0.2 1"/>
-        </material>
+        <visual>
+            <geometry>
+                <mesh filename="package://ahand_description/meshes/base_link.STL"/>
+            </geometry>
+            <origin rpy="0 0 0" xyz="0 0 0 "/>
+            <material name="black">
+                <color rgba="0.2 0.2 0.2 1"/>
+            </material>
         </visual>
+        <collision>
+            <origin rpy="0 0 0" xyz="-0.009300 0 -${palm_link_z/2}"/>
+            <geometry>
+                <box size="0.0408 0.1130 ${palm_link_z}"/>
+            </geometry>
+        </collision>
+        <inertial>
+          <origin xyz="0 0 ${palm_link_z/2}" rpy="0 0 0"/>
+          <mass value="0.4154"/>
+          <inertia
+              ixx="1e-4" ixy="0.0" ixz="0.0"
+              iyy="1e-4" iyz="0.0"
+              izz="1e-4"/>
+        </inertial>
     </link>
     <!-- ============================================================================= -->
@@ -97,5 +83,5 @@
     <!-- for LEFT HAND switch the sign of the **offset_origin_y** and **finger_angle_r** parameters-->
     <xacro:finger
-	    name="${name}"
+            name="${name}"
             finger_num="0"
             offset_origin_x="${offset_origin_x_const}"
@@ -105,5 +91,5 @@
             />
     <xacro:finger
-	    name="${name}"
+            name="${name}"
             finger_num="1"
             offset_origin_x="${offset_origin_x_const}"
@@ -113,5 +99,5 @@
             />
     <xacro:finger
-	    name="${name}"
+            name="${name}"
             finger_num="2"
             offset_origin_x="${offset_origin_x_const}"
@@ -122,5 +108,5 @@
     <!-- THUMB -->
     <xacro:thumb_right
-	    name="${name}"
+            name="${name}"
             finger_num="3"
             offset_origin_x="-0.0182"
@@ -131,28 +117,33 @@
             finger_angle_y="-${90*DEG2RAD}"
             />
-      <!--finger_angle_p="-${95*DEG2RAD}"
-      finger_angle_y="-${90*DEG2RAD}"-->
+    </xacro:macro>
     <!-- ============================================================================= -->
-    <xacro:ahand_gazebo name="${name}"/>
-    <xacro:ahand_transmission name="${name}"/>
-   </xacro:macro>
     <!-- THUMB MACRO -->
-   <xacro:macro name="thumb_right" params="name finger_num offset_origin_x offset_origin_y offset_origin_z finger_angle_r finger_angle_p finger_angle_y">
+    <xacro:macro name="thumb_right"
+                 params="name finger_num offset_origin_x offset_origin_y offset_origin_z finger_angle_r finger_angle_p finger_angle_y">
         <!-- [LINK 12] -->
         <link name="${name}_link_${finger_num*4+0}">
-            <inertial>
-              <origin xyz="${-link0_t_x/2} 0 0"/>
-              <xacro:cuboid_inertia_def width="0.02" height="0.04" length="0.04" mass="${thumb_0_mass}"/>
-              <mass value="${thumb_0_mass}" />
-            </inertial>
-            <visual>
-              <geometry>
-                <mesh filename="package://ahand_description/meshes/link_12_right.dae"/>
-              </geometry>
-              <material name="black">
-                <color rgba=".2 .2 .2 1"/>
-              </material>
-              <origin rpy="${180*DEG2RAD} 0 0" xyz="0 0 0"/>
-            </visual>
+            <visual>
+                <geometry>
+                    <mesh filename="package://ahand_description/meshes/link_12.0_right.STL"/>
+                </geometry>
+                <material name="black">
+                    <color rgba=".2 .2 .2 1"/>
+                </material>
+                <origin rpy="${180*DEG2RAD} 0 0" xyz="0 0 0"/>
+            </visual>
+            <collision>
+                <geometry>
+                    <box size="${link0_t_x} ${link0_t_y} ${link0_t_z}"/>
+                </geometry>
+                <origin rpy="0 0 0" xyz="${-0.0358/2+0.0} ${.018/2} ${.029/2}"/>
+            </collision>
+            <inertial>
+              <mass value="0.0176" />
+              <origin xyz="0 0 0" rpy="0 0 0"/>
+              <inertia ixx="1.89273333333e-5" ixy="7.16716e-06" ixz="5.35568e-06"
+                       iyy="1.43008213333e-05" iyz="6.8068e-06"
+                       izz="1.89273333333e-05" />
+            </inertial>
         </link>
         <joint name="${name}_joint_${finger_num*4+0}" type="revolute">
@@ -165,16 +156,11 @@
             <origin rpy="${finger_angle_r} ${finger_angle_p} ${finger_angle_y}"
                     xyz="${offset_origin_x} ${offset_origin_y} ${offset_origin_z}"/>
-            <dynamics damping="${b}" friction="${c}"/>
+            <dynamics damping="3" friction="10"/>
         </joint>
         <!-- [LINK 13] -->
         <link name="${name}_link_${finger_num*4+1}">
-          <inertial>
-            <origin xyz="0.0 0.0 ${link1_t_z/2} "/>
-            <xacro:cuboid_inertia_def width="0.02" height="0.02" length="0.02" mass="${thumb_1_mass}"/>
-            <mass value="${thumb_1_mass}" />
-          </inertial>
-          <visual>
-                <geometry>
-                    <mesh filename="package://ahand_description/meshes/link_13.dae"/>
+            <visual>
+                <geometry>
+                    <mesh filename="package://ahand_description/meshes/link_13.0.STL"/>
                 </geometry>
                 <material name="black">
@@ -182,4 +168,17 @@
                 </material>
             </visual>
+            <collision>
+                <geometry>
+                    <box size="${links_x} ${links_y} ${link1_t_z}"/>
+                </geometry>
+                <origin rpy="0 0 0" xyz="0 0 ${link1_t_z/2}"/>
+            </collision>
+            <inertial>
+              <mass value="0.0119" />
+              <origin xyz="0 0 0" rpy="0 0 0"/>
+              <inertia ixx="4.24250866667e-06" ixy="1.032087e-06" ixz="1.603525e-06"
+                       iyy="4.52362633333e-06" iyz="1.44808125e-06"
+                       izz="4.24250866667e-06" />
+            </inertial>
         </link>
         <joint name="${name}_joint_${finger_num*4+1}" type="revolute">
@@ -191,17 +190,11 @@
             <child link="${name}_link_${finger_num*4+1}"/>
             <origin xyz="-0.027 0.005 0.0399"/>
-            <dynamics damping="${b}" friction="${c}"/>
+            <dynamics damping="3" friction="5"/>
         </joint>
         <!-- [LINK 14] -->
         <link name="${name}_link_${finger_num*4+2}">
-            <inertial>
-                  <origin xyz="${link2_t_z/2} 0.0 0.0"/>
-                        <xacro:cuboid_inertia_def width="0.02" height="0.02" length="0.02" mass="${thumb_2_mass}"/>
-                  <mass value="${thumb_2_mass}" />
-            </inertial>
-            <visual>
-            	<origin xyz="0 0 0" rpy="${90*DEG2RAD} 0 ${90*DEG2RAD}"/>
-		<geometry>
-                    <mesh filename="package://ahand_description/meshes/link_14.dae"/>
+            <visual>
+                <geometry>
+                    <mesh filename="package://ahand_description/meshes/link_14.0.STL"/>
                 </geometry>
                 <material name="black">
@@ -212,9 +205,15 @@
                     <box size="${links_x} ${links_y} ${link2_t_z}"/>
                 </geometry>
-                <origin rpy="${90*DEG2RAD} 0 ${90*DEG2RAD}" xyz="${link2_t_z/2} 0 0"/>
-            </collision>
+                <origin rpy="0 0 0" xyz="0 0 ${link2_t_z/2}"/>
+            </collision>
+            <inertial>
+              <mass value="0.038" />
+              <origin xyz="0 0 0" rpy="0 0 0"/>
+              <inertia ixx="4.30439933333e-05" ixy="9.57068e-06" ixz="5.1205e-06" iyy="1.44451933333e-05"
+                       iyz="1.342825e-05" izz="4.30439933333e-05" />
+            </inertial>
         </link>
         <joint name="${name}_joint_${finger_num*4+2}" type="revolute">
-            <axis xyz="0 0 -1"/>
+            <axis xyz="0 1 0"/>
             <limit effort="15" velocity="7"
                    lower="${limit_2_t_low+joint_safety_margin}"
@@ -222,18 +221,12 @@
             <parent link="${name}_link_${finger_num*4+1}"/>
             <child link="${name}_link_${finger_num*4+2}"/>
-            <origin xyz="0 0 ${link1_t_z}" rpy="${180*DEG2RAD} -${90*DEG2RAD} -${90*DEG2RAD}"/>
-            <dynamics damping="${b}" friction="${c}"/>
+            <origin xyz="0 0 ${link1_t_z}"/>
+            <dynamics damping="3" friction="10"/>
         </joint>
         <!-- [LINK 15] -->
         <link name="${name}_link_${finger_num*4+3}">
-          <inertial>
-                <origin xyz="${link3_t_z/2} 0.0 0.0"/>
-                      <xacro:cuboid_inertia_def width="0.02" height="0.02" length="0.02" mass="${thumb_3_mass}"/>
-                <mass value="${thumb_3_mass}" />
-          </inertial>
-          <visual>
-            	<origin xyz="0 0 0" rpy="${90*DEG2RAD} 0 ${90*DEG2RAD}"/>
-                <geometry>
-                    <mesh filename="package://ahand_description/meshes/link_15.dae"/>
+            <visual>
+                <geometry>
+                    <mesh filename="package://ahand_description/meshes/link_15.0.STL"/>
                 </geometry>
                 <material name="black">
@@ -242,11 +235,18 @@
             <collision>
                 <geometry>
-                    <box size="${links_x} ${links_y} ${link3_t_z-2.0*fingerTip_r}"/>
-                </geometry>
-                <origin rpy="${90*DEG2RAD} 0 ${90*DEG2RAD}" xyz="${(link3_t_z-2.0*fingerTip_r)/2} 0 0"/>
-            </collision>
+                    <box size="${links_x} ${links_y} ${link3_t_z-fingerTip_r}"/>
+                </geometry>
+                <origin rpy="0 0 0" xyz="0 0 ${(link3_t_z-fingerTip_r)/2}"/>
+            </collision>
+            <inertial>
+              <mass value="0.0388" />
+              <origin xyz="0 0 0" rpy="0 0 0"/>
+              <inertia ixx="3.29223173333e-05" ixy="8.042076e-06" ixz="5.2283e-06"
+                       iyy="1.47493026667e-5" iyz="1.1283525e-5"
+                       izz="3.29223173333e-05" />
+            </inertial>
         </link>
         <joint name="${name}_joint_${finger_num*4+3}" type="revolute">
-            <axis xyz="0 0 -1"/>
+            <axis xyz="0 1 0"/>
             <limit effort="15" velocity="7"
                    lower="${limit_3_t_low+joint_safety_margin}"
@@ -254,16 +254,10 @@
             <parent link="${name}_link_${finger_num*4+2}"/>
             <child link="${name}_link_${finger_num*4+3}"/>
-            <origin xyz="${link2_t_z} 0 0" rpy="0 0 0"/>
-            <dynamics damping="${b}" friction="${c}"/>
-        </joint>
-        <!-- [FINGER TIP THUMB] -->
+            <origin xyz="0 0 ${link2_t_z}"/>
+            <dynamics damping="3" friction="12"/>
+        </joint>
+        <!-- [FINGER TIP] -->
         <link name="${name}_link_${finger_num*4+3}_tip">
-          <inertial>
-                <origin xyz="0.0 0.0 0.0"/>
-                      <xacro:cuboid_inertia_def width="0.02" height="0.05" length="0.02" mass="${thumb_tip_mass}"/>
-                <mass value="${thumb_tip_mass}" />
-          </inertial>
-            <visual>
-                <origin xyz="0 0 0" rpy="${90*DEG2RAD} 0 ${90*DEG2RAD}"/>
+            <visual>
                 <geometry>
                     <mesh filename="package://ahand_description/meshes/link_15.0_tip.STL"/>
@@ -274,30 +268,32 @@
             </visual>
             <collision>
-                <origin xyz="0 0 0" rpy="${90*DEG2RAD} 0 ${90*DEG2RAD}"/>
-                <geometry>
-                    <mesh filename="package://ahand_description/meshes/link_15.0_tip.STL"/>
-                </geometry>
-            </collision>
-        </link>
-        <joint name="${name}_joint_${finger_num*4+3}_tip" type="fixed">
+                <geometry>
+                    <sphere radius="${fingerTip_r}"/>
+                </geometry>
+                <origin rpy="0 0 0" xyz="0 0 0"/>
+            </collision>
+            <inertial>
+              <mass value="0.0168" />
+              <origin xyz="0 0 0" rpy="0 0 0"/>
+              <inertia ixx="9.68e-07" ixy="0" ixz="0"
+                       iyy="9.68e-07" iyz="0"
+                       izz="9.68e-07" />
+            </inertial>
+        </link>
+        <joint name="joint_${finger_num*4+3}_tip" type="fixed">
             <parent link="${name}_link_${finger_num*4+3}"/>
             <child link="${name}_link_${finger_num*4+3}_tip"/>
-            <origin rpy="0 0 0" xyz="${link3_t_z-fingerTip_r} 0 0"/>
+            <origin rpy="0 0 0" xyz="0 0 ${link3_t_z-fingerTip_r}"/>
         </joint>
     </xacro:macro>
     <!-- END THUMB MACRO -->
     <!-- THREE FINGER MACRO -->
-    <xacro:macro name="finger" params="name finger_num offset_origin_x offset_origin_y offset_origin_z finger_angle_r">
+    <xacro:macro name="finger"
+                 params="name finger_num offset_origin_x offset_origin_y offset_origin_z finger_angle_r">
         <!-- [LINK 0, 4, 8] -->
         <link name="${name}_link_${finger_num*4+0}">
-            <inertial>
-              <origin xyz="0.00 0 0.01"/>
-              <xacro:cuboid_inertia_def width="0.025" height="0.02" length="0.025" mass="${link_0_mass}"/>
-              <mass value="${link_0_mass}" />
-            </inertial>
-            <visual>
-                <origin xyz="0 0 0" rpy="0 0 0"/>
-                <geometry>
-                    <mesh filename="package://ahand_description/meshes/link_0.dae"/>
+            <visual>
+                <geometry>
+                    <mesh filename="package://ahand_description/meshes/link_0.0.STL"/>
                 </geometry>
                 <material name="black"/>
@@ -309,4 +305,11 @@
                 <origin rpy="0 0 0" xyz="0 0 ${link0_z/2}"/>
             </collision>
+            <inertial>
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
Commit message: fixed right urdf file

File: ahand_description/urdf/ahand.xacro (robot description, xacro)
@@ -1,6 +1,9 @@
 <?xml version="1.0"?>
 <robot name="ahand" xmlns:xacro="http://ros.org/wiki/xacro">
-    <xacro:property name="hand_type" default="left" />
-    <xacro:include filename="$(find ahand_description)/urdf/ahand_${hand_type}.xacro"/>
+    <xacro:arg name="hand_type" default="right"/>
+    <!-- <xacro:property name="hand_type" default="right" /> -->
+    <xacro:property name="hand_type" default="$(arg hand_type)" />
+    <xacro:include filename="$(find ahand_description)/urdf/ahand_$(arg hand_type).xacro"/>
+    <!-- <xacro:include filename="$(find ahand_description)/urdf/ahand_right.xacro"/> -->
     <link name="world"/>
     <xacro:ahand_robot name="ahand" parent_link="world" xyz="0.0 0 0.15" rpy="0 0 0"/>

File: ahand_description/urdf/ahand_right.xacro (robot description, xacro)
@@ -1,4 +1,4 @@
 <?xml version="1.0"?>
-<robot xmlns:xacro="http://www.ros.org/wiki/xacro" name="ahand_right">
+<robot xmlns:xacro="http://www.ros.org/wiki/xacro" name="right">
     <xacro:property name="DEG2RAD" value="0.01745329251"/>
     <!-- ======================== BASE PARAMS ========================= -->
@@ -45,4 +45,11 @@
     <xacro:property name="limit_3_t_low" value="-0.262"/>
     <!-- ============================================================================= -->
+    <xacro:include filename="$(find ahand_description)/urdf/common.xacro"/>
+    <xacro:property name="b" value="0.2"/>
+    <xacro:property name="c" value="0.0"/>
+    <!-- Include transmissions -->
+    <xacro:include filename="$(find ahand_description)/urdf/ahand_transmission.xacro"/>
+    <!-- Include Gazebo -->
+    <xacro:include filename="$(find ahand_description)/urdf/ahand_gazebo.xacro"/>
     <!-- Base link -->
     <xacro:macro name="ahand_robot" params="name parent_link xyz rpy">
@@ -117,4 +124,6 @@
             finger_angle_y="-${90*DEG2RAD}"
             />
+    <xacro:ahand_gazebo name="${name}"/>
+    <xacro:ahand_transmission name="${name}"/>
     </xacro:macro>
     <!-- ============================================================================= -->
@@ -131,5 +140,5 @@
                     <color rgba=".2 .2 .2 1"/>
                 </material>
-                <origin rpy="${180*DEG2RAD} 0 0" xyz="0 0 0"/>
+                <origin rpy="${0*DEG2RAD} 0 0" xyz="0 0 0"/>
             </visual>
             <collision>
